File: expansion/GfxV9990/Video.sch (KiCad schematic (older format))
At the start: 0 parts

Commit message: Added XCA2075M to library
Parts:
- added U?: CXA2075M, Package_SO:SOP-24_7.5x15.4mm_P1.27mm, symbol Ddraig:CXA2075M
Changed lines of the file:
@@
 Comment4 ""
 $EndDescr
+$Comp
+L Ddraig:CXA2075M U?
+U 1 1 61254DB4
+P 4250 2450
+F 0 "U?" H 4250 3531 50  0000 C CNN
+F 1 "CXA2075M" H 4250 3440 50  0000 C CNN
+F 2 "Package_SO:SOP-24_7.5x15.4mm_P1.27mm" H 4250 2450 50  0001 C CNN
+F 3 "" H 4250 2450 50  0001 C CNN
+	1    4250 2450
+	1    0    0    -1
+$EndComp
 $EndSCHEMATC
