File: expansion/GfxFPGAS3/FPGA.sch (KiCad schematic (older format))
At the start: 15 parts, among them U301 XC3S500E-4PQG208I, U302 W25Q64JVSSIM

Commit message: Working on the pinning of the FPGA pins
Connections:
- net A1: now also U301.86 (IO_12P_2/M0)
- net A10: now also U301.75 (IO_L08N_2/DD/GCLK13)
- net A11: now also U301.74 (IO_L08P_2/D7/GCLK12)
- net A12: now also U301.69 (IO_L06N_2)
- net A13: now also U301.68 (IO_L06P_2)
- net A14: now also U301.65 (IO_L05N_2)
- net A15: now also U301.64 (IO_L05P_2)
- net A16: now also U301.63 (IO_L04N_2)
- net A17: now also U301.62 (IO_L04P_2)
- net A18: now also U301.61 (IO_L03N_2/MOSI/CSI_B)
- net A19: now also U301.60 (IO_L03P_2/DOUT/BUSY)
- net A2: now also U301.84 (IO/M1)
- net A3: now also U301.83 (IO_L11N_2/D1/GCLK3)
- net A4: now also U301.82 (IO_L11P_2/D2/GCLK2)
- net A5: now also U301.81 (IP_L10N_2/M2/GCLK1)
- net A6: now also U301.80 (IP_L10P_2/RDWR_B/GCLK0)
- net A7: now also U301.78 (IO_L09N_2/D3/GCLK15)
- net A8: now also U301.77 (IO_L09P_2/D4/GCLK14)
- net A9: now also U301.76 (IO/D5)
- net B0: now also U301.128 (IO_L08P_1/A8/RHCLK2); no longer U301.129 (IO_L08N_1/A7/RHCLK3/TRDY1)
- net B1: now also U301.127 (IO_L07N_1/A9/RHCLK1); no longer U301.128 (IO_L08P_1/A8/RHCLK2)
- net B2: now also U301.126 (IO_L07P_1/A10/RHCLK0); no longer U301.127 (IO_L07N_1/A9/RHCLK1)
- net B3: now also U301.123 (IO_L06N_1/VREF_1); no longer U301.126 (IO_L07P_1/A10/RHCLK0)
- net B4: now also U301.122 (IO_L06P_1); no longer U301.123 (IO_L06N_1/VREF_1)
- net B5: now also U301.120 (IO_L05N_1/A11); no longer U301.122 (IO_L06P_1)
- net B6: now also U301.119 (IO_L05P_1/A12); no longer U301.120 (IO_L05N_1/A11)
- net B7: now also U301.116 (IO_L04N_1); no longer U301.119 (IO_L05P_1/A12)
- net D0: now also U301.109 (IO_L02N_1/A13)
- net D1: now also U301.108 (IO_L02P_1/A14)
- net D10: now also U301.96 (IO_L15P_2/A21)
- net D11: now also U301.94 (IO_L14N_2/A22)
- net D12: now also U301.93 (IO_L14P_2/A23)
- net D13: now also U301.90 (IO_L13N_2)
- net D14: now also U301.89 (IO_L13P_2)
- net D15: now also U301.87 (IO_12N_2/DIN/D0)
- net D2: now also U301.107 (IO_L01N_1/A15)
- net D3: now also U301.106 (IO_L01P_1/A16)
- net D4: now also U301.103 (IO_L17N_2/CCLK)
- net D5: now also U301.102 (IO_L17P_2/VS0/A17)
- net D6: now also U301.100 (IO_L16N_2/VS1/A18)
- net D7: now also U301.99 (IO_L16P_2/VS2/A19)
- net D8: now also U301.98 (IO/VREF_2)
- net D9: now also U301.97 (IO_L15N_2/A20)
- net HSYNC: now also U301.112 (IO_L03P_1)
- net PIXELCLOCK: now also U301.115 (IO_L04P_1)
- net SRAM_A0: now also U301.200 (IO_L14N_0/VREF_0)
- net SRAM_A1: now also U301.202 (IO_L15P_0)
- net SRAM_A10: now also U301.164 (IO_L03P_0)
- net SRAM_A11: now also U301.163 (IO_L02N_0/VREF)
- net SRAM_A12: now also U301.162 (IO_L02P_0)
- net SRAM_A13: now also U301.161 (IO_L01N_0)
- net SRAM_A14: now also U301.160 (IO_L01P_0)
- net SRAM_A15: now also U301.177 (IO_L07P_0/GCLK4)
- net SRAM_A16: now also U301.178 (IO_L07N_0/GCLK5)
- net SRAM_A17: now also U301.179 (IO/VREF_0)
- net SRAM_A18: now also U301.180 (IO_L08P_0/GCLK6)
- net SRAM_A19: now also U301.181 (IO_L08N_0/GCLK7)
- net SRAM_A2: now also U301.203 (IO_L15N_0)
- net SRAM_A3: now also U301.205 (IO_L16P_0)
- net SRAM_A4: now also U301.206 (IO_L16N_0/HSWAP)
- net SRAM_A5: now also U301.29 (IO_L09N_3/LHCLK5)
- net SRAM_A6: now also U301.28 (IO_L09P_3/LHCLK3/TRDY2)
- net SRAM_A7: now also U301.25 (IO_L08N_3/LHCLK3/IRDY2)
- net SRAM_A8: now also U301.24 (IO_L08P_3/LHCLK2)
- net SRAM_A9: now also U301.165 (IO_L03N_0)
- net VSYNC: now also U301.113 (IO_L03N_1/VREF)
- net ~BLANK: now also U301.129 (IO_L08N_1/A7/RHCLK3/TRDY1)
- net ~SRAM_CS: now also U301.199 (IO_L14P_0)
- net ~SRAM_LB0: now also U301.31 (IO_L10N_3/LHCLK7)
- net ~SRAM_LB1: now also U301.22 (IO_L07P_3/LHCLK0)
- net ~SRAM_UB0: now also U301.30 (IO_L10P_3/LHCLK6)
- net ~SRAM_UB1: now also U301.23 (IO_L07N_3/LHCLK1)
- net ~SRAM_WE: now also U301.185 (IO_L10P_0/GCLK10)
- net SRAM_D24: now reaches U301.167 (IO_L04P_0)
- net SRAM_D25: now reaches U301.168 (IO_L04N_0/VREF_0)
- net SRAM_D26: now reaches U301.171 (IO_L05P_0)
- net SRAM_D27: now reaches U301.172 (IO_L05N_0)
- net SRAM_D23: now reaches U301.186 (IO_L10N_0/GCLK11)
- net SRAM_D22: now reaches U301.187 (IO)
- net SRAM_D21: now reaches U301.189 (IO_L11P_0)
- net SRAM_D20: now reaches U301.190 (IO_L11N_0)
- net SRAM_D19: now reaches U301.192 (IO_L12P_0)
- net SRAM_D18: now reaches U301.193 (IO_L12N_0/VREF_0)
- net SRAM_D17: now reaches U301.196 (IO_L13P_0)
- net SRAM_D16: now reaches U301.197 (IO_L13N_0)
- net SRAM_D6: now reaches U301.11 (IO_L04P_3)
- net SRAM_D7: now reaches U301.12 (IO_L03N_3)
- net SRAM_D28: now reaches U301.15 (IO_L05P_3)
- net SRAM_D29: now reaches U301.16 (IO_L05N_3)
- net SRAM_D30: now reaches U301.18 (IO_L06P_3)
- net SRAM_D31: now reaches U301.19 (IO_L06N_3)
- net SRAM_D0: now reaches U301.2 (IO_L01P_3)
- net SRAM_D1: now reaches U301.3 (IO_L01N_3)
- net SRAM_D15: now reaches U301.33 (IO_L11P_3)
- net SRAM_D14: now reaches U301.34 (IO_L11N_3)
- net SRAM_D13: now reaches U301.35 (IO_L12P_3)
- net SRAM_D12: now reaches U301.36 (IO_L12N_3)
- net SRAM_D11: now reaches U301.39 (IO_L13P_3)
- net SRAM_D2: now reaches U301.4 (IO_L02P_3)
- net SRAM_D10: now reaches U301.40 (IO_L13N_3)
- net SRAM_D9: now reaches U301.41 (IO_L14P_3)
- net SRAM_D8: now reaches U301.42 (IO_L14N_3)
- net SRAM_D3: now reaches U301.5 (IO_L02N_3/VREF)
- net SRAM_D4: now reaches U301.8 (IO_L03P_3)
- net SRAM_D5: now reaches U301.9 (IO_L03N_P)

Commit message: Some updates to the VGA FPGA pinout
Connections:
- net A1: now also U301.84 (IO/M1); no longer U301.86 (IO_12P_2/M0)
- net A10: now also U301.74 (IO_L08P_2/D7/GCLK12); no longer U301.75 (IO_L08N_2/DD/GCLK13)
- net A11: now also U301.69 (IO_L06N_2); no longer U301.74 (IO_L08P_2/D7/GCLK12)
- net A12: now also U301.72 (IP_L07N_2/VREF); no longer U301.69 (IO_L06N_2)
- net A13: now also U301.71 (IP_L07P_2); no longer U301.68 (IO_L06P_2)
- net A14: now also U301.68 (IO_L06P_2); no longer U301.65 (IO_L05N_2)
- net A15: now also U301.65 (IO_L05N_2); no longer U301.64 (IO_L05P_2)
- net A16: now also U301.64 (IO_L05P_2); no longer U301.63 (IO_L04N_2)
- net A18: now also U301.63 (IO_L04N_2); no longer U301.61 (IO_L03N_2/MOSI/CSI_B)
- net A19: now also U301.58 (IO_L01n_2); no longer U301.60 (IO_L03P_2/DOUT/BUSY)
- net A2: now also U301.83 (IO_L11N_2/D1/GCLK3); no longer U301.84 (IO/M1)
- net A3: now also U301.82 (IO_L11P_2/D2/GCLK2); no longer U301.83 (IO_L11N_2/D1/GCLK3)
- net A4: now also U301.81 (IP_L10N_2/M2/GCLK1); no longer U301.82 (IO_L11P_2/D2/GCLK2)
- net A5: now also U301.80 (IP_L10P_2/RDWR_B/GCLK0); no longer U301.81 (IP_L10N_2/M2/GCLK1)
- net A6: now also U301.78 (IO_L09N_2/D3/GCLK15); no longer U301.80 (IP_L10P_2/RDWR_B/GCLK0)
- net A7: now also U301.77 (IO_L09P_2/D4/GCLK14); no longer U301.78 (IO_L09N_2/D3/GCLK15)
- net A8: now also U301.76 (IO/D5); no longer U301.77 (IO_L09P_2/D4/GCLK14)
- net A9: now also U301.75 (IO_L08N_2/DD/GCLK13); no longer U301.76 (IO/D5)
- net D10: now also U301.94 (IO_L14N_2/A22); no longer U301.96 (IO_L15P_2/A21)
- net D11: now also U301.93 (IO_L14P_2/A23); no longer U301.94 (IO_L14N_2/A22)
- net D12: now also U301.90 (IO_L13N_2); no longer U301.93 (IO_L14P_2/A23)
- net D13: now also U301.89 (IO_L13P_2); no longer U301.90 (IO_L13N_2)
- net D14: now also U301.87 (IO_12N_2/DIN/D0); no longer U301.89 (IO_L13P_2)
- net D15: now also U301.86 (IO_12P_2/M0); no longer U301.87 (IO_12N_2/DIN/D0)
- net D4: now also U301.102 (IO_L17P_2/VS0/A17); no longer U301.103 (IO_L17N_2/CCLK)
- net D5: now also U301.100 (IO_L16N_2/VS1/A18); no longer U301.102 (IO_L17P_2/VS0/A17)
- net D6: now also U301.99 (IO_L16P_2/VS2/A19); no longer U301.100 (IO_L16N_2/VS1/A18)
- net D7: now also U301.98 (IO/VREF_2); no longer U301.99 (IO_L16P_2/VS2/A19)
- net D8: now also U301.97 (IO_L15N_2/A20); no longer U301.98 (IO/VREF_2)
- net D9: now also U301.96 (IO_L15P_2/A21); no longer U301.97 (IO_L15N_2/A20)
- new net CLK_25MHZ: U301.103 (IO_L17N_2/CCLK)
Other:
- moved on the sheet: R301, R302, R303, U301F, U302
Changed lines of the file:
@@
 $Descr A3 16535 11693
 encoding utf-8
-Sheet 5 5
+Sheet 4 5
 Title ""
 Date ""
@@
 L Ddraig:XC3S500E-4PQG208I U301
 U 6 1 61236505
-P 15300 7600
-F 0 "U301" H 15200 8150 50  0000 L CNN
-F 1 "XC3S500E-4PQG208I" H 14950 7100 50  0000 L CNN
-F 2 "Ddraig:QFP50P3060X3060X409-208N" H 15850 7750 50  0001 C CNN
-F 3 "" H 15850 7750 50  0001 C CNN
-	6    15300 7600
+P 15150 9300
+F 0 "U301" H 15050 9850 50  0000 L CNN
+F 1 "XC3S500E-4PQG208I" H 14800 8800 50  0000 L CNN
+F 2 "Ddraig:QFP50P3060X3060X409-208N" H 15700 9450 50  0001 C CNN
+F 3 "" H 15700 9450 50  0001 C CNN
+	6    15150 9300
 	1    0    0    -1
 $EndComp
@@
 Text HLabel 10250 8250 2    50   Input ~ 0
 HOST_CLK
-Text Label 9450 4150 2    50   ~ 0
+Text Label 9450 4050 2    50   ~ 0
 A1
-Text Label 9450 4050 2    50   ~ 0
+Text Label 9450 3950 2    50   ~ 0
 A2
-Text Label 9450 3950 2    50   ~ 0
+Text Label 9450 3850 2    50   ~ 0
 A3
-Text Label 9450 3850 2    50   ~ 0
+Text Label 9450 6250 2    50   ~ 0
 A4
-Text Label 9450 6250 2    50   ~ 0
+Text Label 9450 6150 2    50   ~ 0
 A5
-Text Label 9450 6150 2    50   ~ 0
+Text Label 9450 3750 2    50   ~ 0
 A6
-Text Label 9450 3750 2    50   ~ 0
+Text Label 9450 3650 2    50   ~ 0
 A7
-Text Label 9450 3650 2    50   ~ 0
+Text Label 9450 3550 2    50   ~ 0
 A8
-Text Label 9450 3550 2    50   ~ 0
+Text Label 9450 3450 2    50   ~ 0
 A9
-Text Label 9450 3450 2    50   ~ 0
+Text Label 9450 3350 2    50   ~ 0
 A10
-Text Label 9450 3350 2    50   ~ 0
+Text Label 9450 3250 2    50   ~ 0
 A11
-Text Label 9450 3250 2    50   ~ 0
+Text Label 9450 6050 2    50   ~ 0
 A12
+Text Label 9450 5950 2    50   ~ 0
+A13
 Text Label 9450 3150 2    50   ~ 0
-A13
+A14
 Text Label 9450 3050 2    50   ~ 0
-A14
+A15
 Text Label 9450 2950 2    50   ~ 0
-A15
-Text Label 9450 2850 2    50   ~ 0
 A16
 Text Label 9450 2750 2    50   ~ 0
 A17
-Text Label 9450 2650 2    50   ~ 0
+Text Label 9450 2850 2    50   ~ 0
 A18
-Text Label 9450 2550 2    50   ~ 0
+Text Label 9450 2450 2    50   ~ 0
 A19
 Text Label 5550 2450 2    50   ~ 0
@@
 Text Label 5550 2150 2    50   ~ 0
 D3
-Text Label 9450 5350 2    50   ~ 0
+Text Label 9450 5250 2    50   ~ 0
 D4
-Text Label 9450 5250 2    50   ~ 0
+Text Label 9450 5150 2    50   ~ 0
 D5
-Text Label 9450 5150 2    50   ~ 0
+Text Label 9450 5050 2    50   ~ 0
 D6
-Text Label 9450 5050 2    50   ~ 0
+Text Label 9450 4950 2    50   ~ 0
 D7
-Text Label 9450 4950 2    50   ~ 0
+Text Label 9450 4850 2    50   ~ 0
 D8
-Text Label 9450 4850 2    50   ~ 0
+Text Label 9450 4750 2    50   ~ 0
 D9
-Text Label 9450 4750 2    50   ~ 0
+Text Label 9450 4650 2    50   ~ 0
 D10
-Text Label 9450 4650 2    50   ~ 0
+Text Label 9450 4550 2    50   ~ 0
 D11
-Text Label 9450 4550 2    50   ~ 0
+Text Label 9450 4450 2    50   ~ 0
 D12
-Text Label 9450 4450 2    50   ~ 0
+Text Label 9450 4350 2    50   ~ 0
 D13
-Text Label 9450 4350 2    50   ~ 0
+Text Label 9450 4250 2    50   ~ 0
 D14
-Text Label 9450 4250 2    50   ~ 0
+Text Label 9450 4150 2    50   ~ 0
 D15
 $Comp
 L Ddraig:W25Q64JVSSIM U302
 U 1 1 612280BD
-P 14500 9600
-F 0 "U302" H 14200 10000 50  0000 C CNN
-F 1 "W25Q64JVSSIM" H 14850 10000 50  0000 C CNN
-F 2 "Ddraig:SOIC127P790X195-8N" H 14500 9600 50  0001 C CNN
-F 3 "" H 14500 9600 50  0001 C CNN
-	1    14500 9600
+P 6250 8950
+F 0 "U302" H 5950 9350 50  0000 C CNN
+F 1 "W25Q64JVSSIM" H 6600 9350 50  0000 C CNN
+F 2 "Ddraig:SOIC127P790X195-8N" H 6250 8950 50  0001 C CNN
+F 3 "" H 6250 8950 50  0001 C CNN
+	1    6250 8950
 	1    0    0    -1
 $EndComp
@@
 L power:+3V3 #PWR0306
 U 1 1 61229369
-P 14500 8850
-F 0 "#PWR0306" H 14500 8700 50  0001 C CNN
-F 1 "+3V3" H 14515 9023 50  0000 C CNN
-F 2 "" H 14500 8850 50  0001 C CNN
-F 3 "" H 14500 8850 50  0001 C CNN
-	1    14500 8850
+P 6250 8200
+F 0 "#PWR0306" H 6250 8050 50  0001 C CNN
+F 1 "+3V3" H 6265 8373 50  0000 C CNN
+F 2 "" H 6250 8200 50  0001 C CNN
+F 3 "" H 6250 8200 50  0001 C CNN
+	1    6250 8200
 	1    0    0    -1
 $EndComp
@@
 L power:GND #PWR0307
 U 1 1 6122A215
-P 14500 10150
-F 0 "#PWR0307" H 14500 9900 50  0001 C CNN
-F 1 "GND" H 14505 9977 50  0000 C CNN
-F 2 "" H 14500 10150 50  0001 C CNN
-F 3 "" H 14500 10150 50  0001 C CNN
-	1    14500 10150
-	1    0    0    -1
-$EndComp
-Wire Wire Line
-	14500 10100 14500 10150
-Wire Wire Line
-	14500 9100 14500 8900
+P 6250 9500
+F 0 "#PWR0307" H 6250 9250 50  0001 C CNN
+F 1 "GND" H 6255 9327 50  0000 C CNN
+F 2 "" H 6250 9500 50  0001 C CNN
+F 3 "" H 6250 9500 50  0001 C CNN
+	1    6250 9500
+	1    0    0    -1
+$EndComp
+Wire Wire Line
+	6250 9450 6250 9500
+Wire Wire Line
+	6250 8450 6250 8250
 $Comp
 L Device:R R303
 U 1 1 6122F7CC
-P 15300 9200
-F 0 "R303" H 15370 9246 50  0000 L CNN
-F 1 "10K" H 15370 9155 50  0000 L CNN
-F 2 "Resistor_SMD:R_0805_2012Metric" V 15230 9200 50  0001 C CNN
-F 3 "~" H 15300 9200 50  0001 C CNN
-	1    15300 9200
+P 7050 8550
+F 0 "R303" H 7120 8596 50  0000 L CNN
+F 1 "10K" H 7120 8505 50  0000 L CNN
+F 2 "Resistor_SMD:R_0805_2012Metric" V 6980 8550 50  0001 C CNN
+F 3 "~" H 7050 8550 50  0001 C CNN
+	1    7050 8550
 	1    0    0    -1
 $EndComp
@@
 L Device:R R302
 U 1 1 6122FF62
-P 13850 9150
-F 0 "R302" H 13920 9196 50  0000 L CNN
-F 1 "10K" H 13920 9105 50  0000 L CNN
-F 2 "Resistor_SMD:R_0805_2012Metric" V 13780 9150 50  0001 C CNN
-F 3 "~" H 13850 9150 50  0001 C CNN
-	1    13850 9150
+P 5600 8500
+F 0 "R302" H 5670 8546 50  0000 L CNN
+F 1 "10K" H 5670 8455 50  0000 L CNN
+F 2 "Resistor_SMD:R_0805_2012Metric" V 5530 8500 50  0001 C CNN
+F 3 "~" H 5600 8500 50  0001 C CNN
+	1    5600 8500
 	1    0    0    -1
 $EndComp
@@
 L Device:R R301
 U 1 1 61230429
-P 13550 9150
-F 0 "R301" H 13620 9196 50  0000 L CNN
-F 1 "10K" H 13620 9105 50  0000 L CNN
-F 2 "Resistor_SMD:R_0805_2012Metric" V 13480 9150 50  0001 C CNN
-F 3 "~" H 13550 9150 50  0001 C CNN
-	1    13550 9150
-	1    0    0    -1
-$EndComp
-Wire Wire Line
-	13550 9000 13550 8900
-Wire Wire Line
-	13550 8900 13850 8900
-Connection ~ 14500 8900
-Wire Wire Line
-	14500 8900 14500 8850
-Wire Wire Line
-	14500 8900 15300 8900
-Wire Wire Line
-	15300 8900 15300 9050
-Wire Wire Line
-	13850 9000 13850 8900
-Connection ~ 13850 8900
-Wire Wire Line
-	13850 8900 14500 8900
-Wire Wire Line
-	13850 9300 13850 9500
-Wire Wire Line
-	13850 9500 14000 9500
-Wire Wire Line
-	13550 9300 13550 9700
-Wire Wire Line
-	13550 9700 14000 9700
-Wire Wire Line
-	15300 9350 15300 9500
-Wire Wire Line
-	15300 9500 15000 9500
-Text Label 15250 9600 0    50   ~ 0
+P 5300 8500
+F 0 "R301" H 5370 8546 50  0000 L CNN
+F 1 "10K" H 5370 8455 50  0000 L CNN
+F 2 "Resistor_SMD:R_0805_2012Metric" V 5230 8500 50  0001 C CNN
+F 3 "~" H 5300 8500 50  0001 C CNN
+	1    5300 8500
+	1    0    0    -1
+$EndComp
+Wire Wire Line
+	5300 8350 5300 8250
+Wire Wire Line
+	5300 8250 5600 8250
+Connection ~ 6250 8250
+Wire Wire Line
+	6250 8250 6250 8200
+Wire Wire Line
+	6250 8250 7050 8250
+Wire Wire Line
+	7050 8250 7050 8400
+Wire Wire Line
+	5600 8350 5600 8250
+Connection ~ 5600 8250
+Wire Wire Line
+	5600 8250 6250 8250
+Wire Wire Line
+	5600 8650 5600 8850
+Wire Wire Line
+	5600 8850 5750 8850
+Wire Wire Line
+	5300 8650 5300 9050
+Wire Wire Line
+	5300 9050 5750 9050
+Wire Wire Line
+	7050 8700 7050 8850
+Wire Wire Line
+	7050 8850 6750 8850
+Text Label 7000 8950 0    50   ~ 0
 FLASH_CLK
-Text Label 15250 9700 0    50   ~ 0
+Text Label 7000 9050 0    50   ~ 0
 FLASH_D0
-Text Label 13450 9600 2    50   ~ 0
+Text Label 5200 8950 2    50   ~ 0
 FLASH_D1
-Text Label 13450 9500 2    50   ~ 0
+Text Label 5200 8850 2    50   ~ 0
 FLASH_CS
 Wire Wire Line
-	13450 9500 13850 9500
-Connection ~ 13850 9500
-Wire Wire Line
-	14000 9600 13450 9600
-Wire Wire Line
-	15000 9600 15250 9600
-Wire Wire Line
-	15000 9700 15250 9700
+	5200 8850 5600 8850
+Connection ~ 5600 8850
+Wire Wire Line
+	5750 8950 5200 8950
+Wire Wire Line
+	6750 8950 7000 8950
+Wire Wire Line
+	6750 9050 7000 9050
 Text HLabel 5350 2550 0    50   Output ~ 0
 HSYNC
@@
 	5850 3650 5350 3650
 Wire Wire Line
+	9450 5150 9700 5150
+Wire Wire Line
 	9450 5250 9700 5250
 Wire Wire Line
-	9450 5350 9700 5350
-Wire Wire Line
 	5550 2150 5850 2150
 Wire Wire Line
@@
 	5550 2450 5850 2450
 Wire Wire Line
+	9450 4150 9700 4150
+Wire Wire Line
 	9450 4250 9700 4250
 Wire Wire Line
@@
 	9450 5050 9700 5050
 Wire Wire Line
-	9450 5150 9700 5150
-Wire Wire Line
-	9700 2550 9450 2550
-Wire Wire Line
-	9700 2650 9450 2650
+	9700 2450 9450 2450
 Wire Wire Line
 	9700 2750 9450 2750
@@
 	9700 3150 9450 3150
 Wire Wire Line
+	9700 5950 9450 5950
+Wire Wire Line
+	9700 6050 9450 6050
+Wire Wire Line
 	9700 3250 9450 3250
 Wire Wire Line
@@
 Wire Wire Line
 	9700 4050 9450 4050
-Wire Wire Line
-	9700 4150 9450 4150
 Wire Wire Line
 	2300 3050 2050 3050
@@
 Wire Wire Line
 	5850 2550 5350 2550
+Text Label 9450 5350 2    50   ~ 0
+CLK_25MHZ
+Wire Wire Line
+	9450 5350 9700 5350
+Text HLabel 10200 8000 0    50   Output ~ 0
+~BUSEN
 $EndSCHEMATC

Commit message: Additional work to FPGA VGA schematic
Parts:
- added C?: 0.1uF, symbol Device:CP
- added D?: LED, symbol Device:LED
- added J?: JTAG, symbol Connector_Generic:Conn_01x06
- added Q?: BC856, Package_TO_SOT_SMD:SOT-23, symbol Transistor_BJT:BC856
- added R? (x5): 10K, symbol Device:R
- added R?: 1K, symbol Device:R
- added R?: 220R, symbol Device:R
- added Y?: ECS-3963, Ddraig:OSC_ECS-3963, symbol Ddraig:ECS-3963
Connections:
- net +3V3: now also J?.1 (Pin_1), Q?.2 (E), R?.1, R?.1, Y?.1 (EN), Y?.4 (VDD)
- net A1: now also R?.1
- net A4: now also R?.1
- net CLK_25MHZ: now also Y?.3 (O/P)
- net D15: now also R?.1
- net GND: now also C?.2, J?.6 (Pin_6), R?.2, R?.2, R?.2, R?.2, Y?.2 (GND)
- net FPGA_INITB: now reaches U301.56 (IO_L01N_2/INIT_B)
- net FPGA_INITB: now also R?.2
- net FPGA_PROGB: now reaches U301.1 (PROG_B)
- net FPGA_PROGB: now also C?.1, R?.2
- net FPGA_DONE: now reaches U301.104 (DONE)
- net FPGA_DONE: now also R?.2
- net at U301.155 (TMS): now also J?.5 (Pin_5)
- net at U301.157 (TDO): now also J?.4 (Pin_4)
- net at U301.158 (TCK): now also J?.2 (Pin_2)
- net at U301.207 (TDI): now also J?.3 (Pin_3)
- new net: Q?.1 (B), R?.1
- new net: D?.2 (A), Q?.3 (C)
- new net: D?.1 (K), R?.1

Commit message: More work on VGA card
Parts:
- removed D?: LED, symbol Device:LED
- removed Q?: BC856, Package_TO_SOT_SMD:SOT-23, symbol Transistor_BJT:BC856
- removed R?: 1K, symbol Device:R
- removed R?: 220R, symbol Device:R
- added D?: LED, symbol Device:LED
- added R?: 390R, symbol Device:R
- R? (x2): value 10K -> 390R
Connections:
- net +3V3: now also R?.1
- net A1: now also R?.1; no longer R?.1
- net A4: now also R?.1; no longer R?.1
- net D15: now also R?.2; no longer R?.1
- net FPGA_DONE: now also R?.1
- net GND: now also D?.1 (K); no longer R?.2
- new net: D?.2 (A), R?.2
Other:
- moved on the sheet: R?, Y?
