File: yddraig68k/power.sch (KiCad schematic (older format))
At the start: 32 parts, among them J201 ATX-24, J202 ExtPWR, J203 PWRLED, SW201 SW_DPST, U201 74HCT74, U202 74HCT74

Commit message: Updated incorrectly labeled component
Parts:
- U201: value 74HCT74 -> 74HCT14
Changed lines of the file:
@@
 P 7550 4750
 F 0 "U201" H 7550 5067 50  0000 C CNN
-F 1 "74HCT74" H 7550 4976 50  0000 C CNN
+F 1 "74HCT14" H 7550 4976 50  0000 C CNN
 F 2 "Package_SO:SO-14_3.9x8.65mm_P1.27mm" H 7550 4750 50  0001 C CNN
 F 3 "74xx/74hc_hct74.pdf" H 7550 4750 50  0001 C CNN
@@
 P 8050 5200
 F 0 "U201" H 8050 5517 50  0000 C CNN
-F 1 "74HCT74" H 8050 5426 50  0000 C CNN
+F 1 "74HCT14" H 8050 5426 50  0000 C CNN
 F 2 "Package_SO:SO-14_3.9x8.65mm_P1.27mm" H 8050 5200 50  0001 C CNN
 F 3 "74xx/74hc_hct74.pdf" H 8050 5200 50  0001 C CNN
@@
 P 7150 5200
 F 0 "U201" H 7150 5517 50  0000 C CNN
-F 1 "74HCT74" H 7150 5426 50  0000 C CNN
+F 1 "74HCT14" H 7150 5426 50  0000 C CNN
 F 2 "Package_SO:SO-14_3.9x8.65mm_P1.27mm" H 7150 5200 50  0001 C CNN
 F 3 "74xx/74hc_hct74.pdf" H 7150 5200 50  0001 C CNN
@@
 P 10550 2300
 F 0 "U201" H 10550 2617 50  0000 C CNN
-F 1 "74HCT74" H 10550 2526 50  0000 C CNN
+F 1 "74HCT14" H 10550 2526 50  0000 C CNN
 F 2 "Package_SO:SO-14_3.9x8.65mm_P1.27mm" H 10550 2300 50  0001 C CNN
 F 3 "74xx/74hc_hct74.pdf" H 10550 2300 50  0001 C CNN
@@
 P 10550 2900
 F 0 "U201" H 10550 3217 50  0000 C CNN
-F 1 "74HCT74" H 10550 3126 50  0000 C CNN
+F 1 "74HCT14" H 10550 3126 50  0000 C CNN
 F 2 "Package_SO:SO-14_3.9x8.65mm_P1.27mm" H 10550 2900 50  0001 C CNN
 F 3 "74xx/74hc_hct74.pdf" H 10550 2900 50  0001 C CNN
@@
 P 10550 1750
 F 0 "U201" H 10550 2067 50  0000 C CNN
-F 1 "74HCT74" H 10550 1976 50  0000 C CNN
+F 1 "74HCT14" H 10550 1976 50  0000 C CNN
 F 2 "Package_SO:SO-14_3.9x8.65mm_P1.27mm" H 10550 1750 50  0001 C CNN
 F 3 "74xx/74hc_hct74.pdf" H 10550 1750 50  0001 C CNN
@@
 P 9650 2350
 F 0 "U201" H 9450 1950 50  0000 C CNN
-F 1 "74HCT74" H 9850 1950 50  0000 C CNN
+F 1 "74HCT14" H 9850 1950 50  0000 C CNN
 F 2 "Package_SO:SO-14_3.9x8.65mm_P1.27mm" H 9650 2350 50  0001 C CNN
 F 3 "74xx/74hc_hct74.pdf" H 9650 2350 50  0001 C CNN

Commit message: Fix for POWER and RESET switches
Parts:
- removed SW201: SW_DPST, Button_Switch_THT:SW_TH_Tactile_Omron_B3F-10xx, symbol Switch:SW_DPST
- added SW201: SW_SPST, Button_Switch_THT:SW_PUSH_6mm_H4.3mm, symbol Switch:SW_SPST
Connections:
- net GND: now also SW201.1 (A)
- net at J202.1 (Pin_1), R201.2, R202.2: now also SW201.2 (B)
Other:
- moved on the sheet: J202
Changed lines of the file:
@@
-$EndComp
-$Comp
-L Switch:SW_DPST SW201
-U 1 1 605A19F0
-P 4600 5400
-F 0 "SW201" H 4600 5725 50  0000 C CNN
-F 1 "SW_DPST" H 4600 5634 50  0000 C CNN
-F 2 "Button_Switch_THT:SW_TH_Tactile_Omron_B3F-10xx" H 4600 5400 50  0001 C CNN
-F 3 "~" H 4600 5400 50  0001 C CNN
-	1    4600 5400
-	0    1    -1   0
 $EndComp
 $Comp
@@
 L Connector_Generic:Conn_01x02 J202
 U 1 1 605A428A
-P 4050 5350
-F 0 "J202" H 4130 5342 50  0000 L CNN
-F 1 "ExtPWR" H 4130 5251 50  0000 L CNN
-F 2 "Connector_PinHeader_2.54mm:PinHeader_1x02_P2.54mm_Vertical" H 4050 5350 50  0001 C CNN
-F 3 "~" H 4050 5350 50  0001 C CNN
-	1    4050 5350
+P 4200 5350
+F 0 "J202" H 4280 5342 50  0000 L CNN
+F 1 "ExtPWR" H 4280 5251 50  0000 L CNN
+F 2 "Connector_PinHeader_2.54mm:PinHeader_1x02_P2.54mm_Vertical" H 4200 5350 50  0001 C CNN
+F 3 "~" H 4200 5350 50  0001 C CNN
+	1    4200 5350
 	-1   0    0    -1
 $EndComp
@@
 $EndComp
 Wire Wire Line
-	4500 5750 4500 5600
-Wire Wire Line
 	4700 5600 4700 5750
 Connection ~ 4700 5750
 Wire Wire Line
-	4700 5750 4500 5750
-Wire Wire Line
 	5000 4600 5000 4750
 Wire Wire Line
 	5000 5050 4700 5050
-Wire Wire Line
-	4500 5050 4500 5200
 Wire Wire Line
 	4700 5200 4700 5050
 Connection ~ 4700 5050
-Wire Wire Line
-	4700 5050 4500 5050
 Wire Wire Line
 	5500 4750 5650 4750
@@
 	4700 5750 5650 5750
 Wire Wire Line
-	4250 5350 4300 5350
-Wire Wire Line
-	4300 5350 4300 5050
-Wire Wire Line
-	4300 5050 4500 5050
-Connection ~ 4500 5050
-Connection ~ 4500 5750
-Wire Wire Line
-	4250 5450 4300 5450
-Wire Wire Line
-	4300 5450 4300 5750
-Wire Wire Line
-	4300 5750 4500 5750
+	4400 5350 4450 5350
+Wire Wire Line
+	4450 5350 4450 5050
+Wire Wire Line
+	4400 5450 4450 5450
+Wire Wire Line
+	4450 5450 4450 5750
 Wire Wire Line
 	9350 4850 9750 4850
+$Comp
+L Switch:SW_SPST SW201
+U 1 1 6125E45F
+P 4700 5400
+F 0 "SW201" V 4746 5312 50  0000 R CNN
+F 1 "SW_SPST" V 4655 5312 50  0000 R CNN
+F 2 "Button_Switch_THT:SW_PUSH_6mm_H4.3mm" H 4700 5400 50  0001 C CNN
+F 3 "~" H 4700 5400 50  0001 C CNN
+	1    4700 5400
+	0    -1   -1   0
+$EndComp
+Wire Wire Line
+	4450 5050 4700 5050
+Wire Wire Line
+	4450 5750 4700 5750
 $EndSCHEMATC

Commit message: FIx for 74HCT74 power symbol connections
Connections:
- net +5V_SB: now also U202.14 (VCC); no longer U202.7 (GND)
- net GND: now also U202.7 (GND); no longer U202.14 (VCC)
Changed lines of the file:
@@
 F 3 "74xx/74hc_hct74.pdf" H 10550 6250 50  0001 C CNN
 	3    10550 6250
-	1    0    0    1
+	1    0    0    -1
 $EndComp
 $Comp
