File: yddraig09/Keyboard.sch (KiCad schematic (older format))
At the start: 0 parts

Commit message: Added some parts for the keyboard controller
Parts:
- added C? (x2): 22pF, symbol Device:C
- added J?: Keyboard, symbol Connector_Generic:Conn_01x20
- added RN?: 10K, Resistor_THT:R_Array_SIP9, symbol Device:R_Network08
- added U?: AT89C51-24PI, symbol Ddraig:AT89C51-24PI
- added U?: IDT7201, symbol Memory_RAM:IDT7201
- added U?: 74LS138, symbol 74xx:74LS138
- added Y?: Crystal, symbol Device:Crystal
Connections:
- new net: C?.1, U?.18 (XTAL2), Y?.2
- new net: C?.1, U?.19 (XTAL1), Y?.1
- new net +5V: J?.4 (Pin_4), RN?.1 (common), U?.40 (VCC)
- new net DB0: U?.9 (Q0)
- new net DB1: U?.10 (Q1)
- new net DB2: U?.11 (Q2)
- new net DB3: U?.12 (Q3)
- new net DB4: U?.16 (Q4)
- new net DB5: U?.17 (Q5)
- new net DB6: U?.18 (Q6)
- new net DB7: U?.19 (Q7)
- new net GND: C?.2, C?.2, J?.1 (Pin_1), U?.2 (D8), U?.20 (GND), U?.31 (~EA~/VPP), U?.7 (XI)
- new net RESET: U?.9 (RESET)
- new net SCDAT0: U?.21 (P2.0(A8)), U?.6 (D0)
- new net SCDAT1: U?.22 (P2.1(A9)), U?.5 (D1)
- new net SCDAT2: U?.23 (P2.2(A10)), U?.4 (D2)
- new net SCDAT3: U?.24 (P2.3(A11)), U?.3 (D3)
- new net SCDAT4: U?.25 (P2.4(A12)), U?.27 (D4)
- new net SCDAT5: U?.26 (D5), U?.26 (P2.5(A13))
- new net SCDAT6: U?.25 (D6), U?.27 (P2.6(A14))
- new net SCDAT7: U?.24 (D7), U?.28 (P2.7(A15))
- new net ~COL0: U?.1 (P1.0)
- new net ~COL1: U?.2 (P1.1)
- new net ~COL2: U?.3 (P1.2)
- new net ~COL4: U?.5 (P1.4)
- new net ~COL5: U?.6 (P1.5)
- new net ~COL6: U?.7 (P1.6)
- new net ~COL7: U?.8 (P1.7)
- new net ~FIFO_CLR: U?.17 (P3.7(~RD~)), U?.22 (CLR)
- new net ~FIFO_WR: U?.1 (WR), U?.16 (P3.6(~WR~))
- new net ~ROW0: RN?.2 (R1), U?.39 (P0.0(AD0))
- new net ~ROW1: RN?.3 (R2), U?.38 (P0.1(AD1))
- new net ~ROW2: RN?.4 (R3), U?.37 (P0.2(AD2))
- new net ~ROW3: RN?.5 (R4), U?.36 (P0.3(AD3))
- new net ~ROW4: RN?.6 (R5), U?.35 (P0.4(AD4))
- new net ~ROW5: RN?.7 (R6), U?.34 (P0.5(AD5))
- new net ~ROW6: RN?.8 (R7), U?.33 (P0.6(AD6))
- new net ~ROW7: U?.32 (P0.7(AD7))
- no-connect marks 0 -> 4
