File: yddraig09/Keyboard.sch (KiCad schematic (older format))
At the start: 8 parts

Commit message: Added RAM/ROM Banking idea
Connections:
- net DB0 renamed D0
- net DB1 renamed D1
- net DB2 renamed D2
- net DB3 renamed D3
- net DB4 renamed D4
- net DB5 renamed D5
- net DB6 renamed D6
- net DB7 renamed D7
Changed lines of the file:
@@
 $Descr A4 11693 8268
 encoding utf-8
-Sheet 9 9
+Sheet 9 11
 Title ""
 Date ""
@@
 Wire Wire Line
 	7300 2750 7300 2650
-Text Label 9000 1850 0    50   ~ 0
-DB0
-Text Label 9000 1950 0    50   ~ 0
-DB1
-Text Label 9000 2050 0    50   ~ 0
-DB2
-Text Label 9000 2150 0    50   ~ 0
-DB3
-Text Label 9000 2250 0    50   ~ 0
-DB4
-Text Label 9000 2350 0    50   ~ 0
-DB5
-Text Label 9000 2450 0    50   ~ 0
-DB6
-Text Label 9000 2550 0    50   ~ 0
-DB7
 Entry Wire Line
 	9400 2650 9300 2550
@@
 	6600 2850 7400 2850
 Text HLabel 9500 2750 2    50   Input ~ 0
-DB[0..7]
+D[0..7]
 Wire Bus Line
 	9400 2750 9500 2750
@@
 	1800 1850 1800 3900
 NoConn ~ 1550 1950
+Text Label 9000 1850 0    50   ~ 0
+D0
+Text Label 9000 1950 0    50   ~ 0
+D1
+Text Label 9000 2050 0    50   ~ 0
+D2
+Text Label 9000 2150 0    50   ~ 0
+D3
+Text Label 9000 2250 0    50   ~ 0
+D4
+Text Label 9000 2350 0    50   ~ 0
+D5
+Text Label 9000 2450 0    50   ~ 0
+D6
+Text Label 9000 2550 0    50   ~ 0
+D7
 Wire Bus Line
 	9400 1950 9400 2750

Commit message: Small updates to keyboard and RAM pages
Parts:
- added R?: 10K, symbol Device:R
- added U?: 74HCT541, symbol 74xx:74HCT541
Connections:
- net +5V: now also U?.16 (VCC), U?.23 (FL), U?.28 (VCC), U?.6 (E3), R?.1, U?.20 (VCC); no longer J?.4 (Pin_4)
- net GND: now also U?.14 (VSS), U?.2 (A1), U?.3 (A2), U?.8 (GND), U?.10 (GND), U?.19 (G2), U?.4 (A2), U?.5 (A3), U?.6 (A4), U?.7 (A5), U?.8 (A6), U?.9 (A7); no longer J?.1 (Pin_1)
- net ~COL3: now also U?.4 (P1.3)
- net ~ROW7: now also RN?.9 (R8)
- net ~COL8: now reaches U?.14 (P3.4(T0))
- net ~ROW8: now reaches U?.15 (P3.5(T1))
- net ~ROW8: now also R?.2
- net ~FIFO_RD: now reaches U?.15 (RD)
- net ~FIFO_RD: now also U?.15 (O0)
- net ~FIFO_EMPTY: now reaches U?.21 (EF)
- net ~FIFO_EMPTY: now also U?.2 (A0)
- net ~FIFO_FULL: now reaches U?.8 (FF)
- net ~FIFO_FULL: now also U?.3 (A1)
- net A0: now reaches U?.1 (A0)
- net at U?.14 (O1): now also U?.1 (G1)
- net ~CS_KBD: now reaches U?.4 (E1)
- net ~RD: now reaches U?.5 (E2)
- net D0 renamed BD0
- net BD0: now also U?.18 (Y0)
- net D1 renamed BD1
- net BD1: now also U?.17 (Y1)
- net D2 renamed BD2
- net BD2: now also U?.16 (Y2)
- net D3 renamed BD3
- net BD3: now also U?.15 (Y3)
- net D4 renamed BD4
- net BD4: now also U?.14 (Y4)
- net D5 renamed BD5
- net BD5: now also U?.13 (Y5)
- net D6 renamed BD6
- net BD6: now also U?.12 (Y6)
- net D7 renamed BD7
- net BD7: now also U?.11 (Y7)
- no-connect marks 4 -> 5
Other:
- moved on the sheet: C?, J?, RN?, U?, Y?

Commit message: More work on 6809 board
Connections:
- net BD0: no longer U?.18 (Y0)
- net BD1: no longer U?.17 (Y1)
- net BD2: no longer U?.16 (Y2)
- net BD3: no longer U?.15 (Y3)
- net BD4: no longer U?.14 (Y4)
- net BD5: no longer U?.13 (Y5)
- net BD6: no longer U?.12 (Y6)
- net BD7: no longer U?.11 (Y7)
- net ~COL0: now also J?.20 (Pin_20)
- net ~COL1: now also J?.19 (Pin_19)
- net ~COL2: now also J?.18 (Pin_18)
- net ~COL3: now also J?.17 (Pin_17)
- net ~COL4: now also J?.16 (Pin_16)
- net ~COL5: now also J?.15 (Pin_15)
- net ~COL6: now also J?.14 (Pin_14)
- net ~COL7: now also J?.13 (Pin_13)
- net ~COL8: now also J?.1 (Pin_1)
- net ~ROW0: now also J?.12 (Pin_12)
- net ~ROW1: now also J?.11 (Pin_11)
- net ~ROW2: now also J?.10 (Pin_10)
- net ~ROW3: now also J?.9 (Pin_9)
- net ~ROW4: now also J?.8 (Pin_8)
- net ~ROW5: now also J?.7 (Pin_7)
- net ~ROW6: now also J?.6 (Pin_6)
- net ~ROW7: now also J?.5 (Pin_5)
- net ~ROW8: now also J?.3 (Pin_3)
- new net D0: U?.18 (Y0)
- new net D1: U?.17 (Y1)
- new net D2: U?.16 (Y2)
- new net D3: U?.15 (Y3)
- new net D4: U?.14 (Y4)
- new net D5: U?.13 (Y5)
- new net D6: U?.12 (Y6)
- new net D7: U?.11 (Y7)
- no-connect marks 5 -> 6

Commit message: More 6809 changes
Parts:
- Y?: value Crystal -> 12Mhz
Other:
- moved on the sheet: C?, J?, R?, RN?, U?, Y?
