File: yddraig09/Audio.kicad_sch (KiCad schematic)
At the start: 42 parts, among them J1 Joystick 2, J2 Joystick 1, J3 Audio Out, U15 YM2203, U16 YM3014B, U17 NE5532

Commit message: Updated yddraig09 silkscreen
Other:
- title: Y Ddraig Fechan -> Y Ddraig Fach
Changed lines of the file:
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@@
   (paper "A4")
   (title_block
-    (title "Y Ddraig Fechan")
+    (title "Y Ddraig Fach")
     (company "Stephen Moody")
   )

Commit message: Considering adding second sound channel to 6809 board
Parts:
- added C104, C105: 100nf, Capacitor_THT:C_Disc_D5.0mm_W2.5mm_P2.50mm, symbol Device:C
- added C106, C107, C108, C109: 10uF, Capacitor_THT:CP_Radial_D5.0mm_P2.50mm, symbol Device:C_Polarized
- added C110: 1.5nF, Capacitor_THT:C_Disc_D5.0mm_W2.5mm_P2.50mm, symbol Device:C
- added J18, J19: Conn_01x10, symbol Connector_Generic:Conn_01x10
- added R55, R56, R57: 1K, Resistor_THT:R_Axial_DIN0207_L6.3mm_D2.5mm_P10.16mm_Horizontal, symbol Device:R
- added R58, R59, R60, R61: 4K7, Resistor_THT:R_Axial_DIN0207_L6.3mm_D2.5mm_P10.16mm_Horizontal, symbol Device:R
- added RV2: 100K, Potentiometer_THT:Potentiometer_Bourns_3386F_Vertical, symbol Device:R_Potentiometer
- added U48: 74LS00, symbol 74xx:74LS00
- added U49: YM2203, Package_DIP:DIP-40_W15.24mm_Socket, symbol Ddraig:YM2203
- added U50: YM3014B, Package_DIP:DIP-8_W7.62mm_Socket, symbol Ddraig:YM3014B
- added U51: NE5532, Package_DIP:DIP-8_W7.62mm_Socket, symbol Amplifier_Operational:NE5532
Connections:
- net +5V: now also J18.1 (Pin_1), J19.1 (Pin_1), U48.14 (VCC), U49.21 (VDD), U50.1 (VDD)
- net A0: now also U49.37 (A0)
- net AUDIO_L: no longer J3.3
- net D0: now also U49.40 (D0)
- net D1: now also U49.2 (D1)
- net D2: now also U49.3 (D2)
- net D3: now also U49.4 (D3)
- net D4: now also U49.5 (D4)
- net D5: now also U49.6 (D5)
- net D6: now also U49.7 (D6)
- net D7: now also U49.8 (D7)
- net GND: now also C104.2, C105.2, C109.2, J18.10 (Pin_10), J19.10 (Pin_10), R55.2, R56.2, R57.2, RV2.3, U48.7 (GND), U49.1 (GND), U49.17 (AGND), U50.6 (GND)
- net SND_CLK: now also U49.38 (CLK-M)
- net ~{CS_SND}: now also U48.1, U48.2; no longer U15.34 (~{CS})
- net ~{IRQ_SND}: now also U49.25 (~{IRQ})
- net ~{RD}: now also U49.36 (~{RD})
- net ~{RESET}: now also U49.24 (~{RESET})
- net ~{WR}: now also U49.35 (~{WR})
- net AUDIO_OUT renamed AUDIO_OUT_L
- new net: C105.1, U50.8 (MP), U51.1, U51.2 (-)
- new net: C109.1, U50.7 (RB), U51.3 (+)
- new net: J19.2 (Pin_2), U49.26 (IOB0)
- new net: J19.3 (Pin_3), U49.27 (IOB1)
- new net: J19.4 (Pin_4), U49.28 (IOB2)
- new net: J19.5 (Pin_5), U49.29 (IOB3)
- new net: J19.6 (Pin_6), U49.30 (IOB4)
- new net: J19.7 (Pin_7), U49.31 (IOB5)
- new net: J19.8 (Pin_8), U49.32 (IOB6)
- new net: J19.9 (Pin_9), U49.33 (IOB7)
- new net: C107.2, R56.1, U49.19 (ANALOGB)
- new net: C108.2, R57.1, U49.20 (ANALOGA)
- new net: C107.1, R60.2
- new net: C104.1, U50.2 (ToBUFF), U51.5 (+)
- new net: C106.1, R59.2
- new net: U48.12, U48.3, U48.9
- new net: U48.13, U48.6
- new net: J18.8 (Pin_8), U49.10 (IOA6)
- new net: J18.7 (Pin_7), U49.11 (IOA5)
- new net: J18.6 (Pin_6), U49.12 (IOA4)
- new net: J18.5 (Pin_5), U49.13 (IOA3)
- new net: J18.4 (Pin_4), U49.14 (IOA2)
- new net: J18.3 (Pin_3), U49.15 (IOA1)
- new net: J18.2 (Pin_2), U49.16 (IOA0)
- new net: C106.2, R55.1, U49.18 (ANALOGC)
- new net: U49.22 (SH), U50.3 (LOAD)
- new net: U49.23 (OP-O), U50.4 (SD)
- new net: U49.39 (CLK-S), U50.5 (CLOCK)
- new net: J18.9 (Pin_9), U49.9 (IOA7)
- new net: C108.1, R61.2
- new net: C110.2, R58.2, U51.6 (-)
- new net A4: U48.10, U48.4, U48.5
- new net AUDIO_OUT_R: C110.1, R58.1, R59.1, R60.1, R61.1, RV2.1, U51.7
- new net AUDIO_R: J3.3, RV2.2
- new net ~{CS_SND1}: U15.34 (~{CS}), U48.11
- new net ~{CS_SND2}: U48.8, U49.34 (~{CS})
Other:
- moved on the sheet: C20, C21, C22, C23, C24, C25, C26, C27, C28, C29, C30, C31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

Commit message: Small updates to 6809 and 030 board, remove old files
Parts:
- removed C104, C105: 100nf, Capacitor_THT:C_Disc_D5.0mm_W2.5mm_P2.50mm, symbol Device:C
- removed C106, C107, C108, C109: 10uF, Capacitor_THT:CP_Radial_D5.0mm_P2.50mm, symbol Device:C_Polarized
- removed C110, C28: 1.5nF, Capacitor_THT:C_Disc_D5.0mm_W2.5mm_P2.50mm, symbol Device:C
- removed J18, J19: Conn_01x10, symbol Connector_Generic:Conn_01x10
- removed R55, R56, R57: 1K, Resistor_THT:R_Axial_DIN0207_L6.3mm_D2.5mm_P10.16mm_Horizontal, symbol Device:R
- removed R58, R59, R6, R60, R61: 4K7, Resistor_THT:R_Axial_DIN0207_L6.3mm_D2.5mm_P10.16mm_Horizontal, symbol Device:R
- removed RV2: 100K, Potentiometer_THT:Potentiometer_Bourns_3386F_Vertical, symbol Device:R_Potentiometer
- removed U48: 74LS00, symbol 74xx:74LS00
- removed U49: YM2203, Package_DIP:DIP-40_W15.24mm_Socket, symbol Ddraig:YM2203
- removed U50: YM3014B, Package_DIP:DIP-8_W7.62mm_Socket, symbol Ddraig:YM3014B
- removed U51: NE5532, Package_DIP:DIP-8_W7.62mm_Socket, symbol Amplifier_Operational:NE5532
- added C17: 1uF, Capacitor_THT:CP_Radial_D5.0mm_P2.50mm, symbol Device:C_Polarized
- added R19, R20: 100R, Resistor_THT:R_Axial_DIN0207_L6.3mm_D2.5mm_P10.16mm_Horizontal, symbol Device:R
- J2: renamed from J1; symbol Connector:DB9_Male_MountingHoles -> Connector:DE9_Plug_MountingHoles
- J3: renamed from J2; symbol Connector:DB9_Male_MountingHoles -> Connector:DE9_Plug_MountingHoles
- RV1: value 100K -> 10K
- renumbered C20 to C11, C21 to C12, C23 to C13, C24 to C14, C25 to C15, C26 to C16, C22 to C18, C27 to C19, C29 to C20, C31 to C21, C30 to C22, J3 to J4, R3 to R12, R4 to R13, R5 to R14, R7 to R15, R8 to R16, R9 to R17, U15 to U5, U16 to U6, U17 to U7
Connections:
- net ~{CS_SND1} is gone; now on net ~{CS_SND}: U5.34 (~{CS})
- net AUDIO_L: now also R19.2; no longer RV1.2
- net AUDIO_R: now also R20.2
- net at U7.6 (-): now also U7.7, C17.1
- net AUDIO_OUT_L renamed AUDIO_OUT
- net AUDIO_OUT: no longer U7.7
- new net: R19.1, R20.1, RV1.2
Other:
- moved on the sheet: C11, C12, C13, C14, C15, C16, C18, C19, C20, C21, C22, J4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
