File: yddraig030/DRAMBuffers.sch (KiCad schematic (older format))
At the start: 7 parts

Commit message: Changes to 6809 and 68030 schematics
Parts:
- gave numbers to parts that had none: 7
Changed lines of the file:
@@
 $Descr A4 11693 8268
 encoding utf-8
-Sheet 3 16
+Sheet 13 15
 Title ""
 Date ""
@@
 ~BCAS_B[0..3]
 $Comp
-L 74xx:74LS241 U?
+L 74xx:74LS241 U1101
 U 1 1 61E721B4
 P 3000 2000
-F 0 "U?" H 2750 2650 50  0000 C CNN
+F 0 "U1101" H 2750 2650 50  0000 C CNN
 F 1 "74LS241" H 3250 2650 50  0000 C CNN
 F 2 "" H 3000 2000 50  0001 C CNN
@@
 CAS_B3
 $Comp
-L 74xx:74LS241 U?
+L 74xx:74LS241 U1102
 U 1 1 61E75709
 P 3000 4250
-F 0 "U?" H 2750 4900 50  0000 C CNN
+F 0 "U1102" H 2750 4900 50  0000 C CNN
 F 1 "74LS241" H 3250 4900 50  0000 C CNN
 F 2 "" H 3000 4250 50  0001 C CNN
@@
 $EndComp
 $Comp
-L 74xx:74LS241 U?
+L 74xx:74LS241 U1103
 U 1 1 61E772F6
 P 3000 6550
-F 0 "U?" H 2750 7200 50  0000 C CNN
+F 0 "U1103" H 2750 7200 50  0000 C CNN
 F 1 "74LS241" H 3250 7200 50  0000 C CNN
 F 2 "" H 3000 6550 50  0001 C CNN
@@
 	10500 1850 10600 1850
 $Comp
-L 74xx:74LS245 U?
+L 74xx:74LS245 U1104
 U 1 1 62039424
 P 6450 2750
-F 0 "U?" H 6200 3400 50  0000 C CNN
+F 0 "U1104" H 6200 3400 50  0000 C CNN
 F 1 "74LS245" H 6650 3400 50  0000 C CNN
 F 2 "" H 6450 2750 50  0001 C CNN
@@
 $EndComp
 $Comp
-L power:GND #PWR?
+L power:GND #PWR01110
 U 1 1 6203E2DE
 P 6450 3600
-F 0 "#PWR?" H 6450 3350 50  0001 C CNN
+F 0 "#PWR01110" H 6450 3350 50  0001 C CNN
 F 1 "GND" H 6455 3427 50  0000 C CNN
 F 2 "" H 6450 3600 50  0001 C CNN
@@
 $EndComp
 $Comp
-L power:+5V #PWR?
+L power:+5V #PWR01109
 U 1 1 6203E83F
 P 6450 1900
-F 0 "#PWR?" H 6450 1750 50  0001 C CNN
+F 0 "#PWR01109" H 6450 1750 50  0001 C CNN
 F 1 "+5V" H 6465 2073 50  0000 C CNN
 F 2 "" H 6450 1900 50  0001 C CNN
@@
 	5850 3250 5950 3250
 $Comp
-L 74xx:74LS245 U?
+L 74xx:74LS245 U1106
 U 1 1 62053D27
 P 9450 2750
-F 0 "U?" H 9200 3400 50  0000 C CNN
+F 0 "U1106" H 9200 3400 50  0000 C CNN
 F 1 "74LS245" H 9650 3400 50  0000 C CNN
 F 2 "" H 9450 2750 50  0001 C CNN
@@
 $EndComp
 $Comp
-L power:GND #PWR?
+L power:GND #PWR01116
 U 1 1 62053D2D
 P 9450 3600
-F 0 "#PWR?" H 9450 3350 50  0001 C CNN
+F 0 "#PWR01116" H 9450 3350 50  0001 C CNN
 F 1 "GND" H 9455 3427 50  0000 C CNN
 F 2 "" H 9450 3600 50  0001 C CNN
@@
 $EndComp
 $Comp
-L power:+5V #PWR?
+L power:+5V #PWR01115
 U 1 1 62053D33
 P 9450 1900
-F 0 "#PWR?" H 9450 1750 50  0001 C CNN
+F 0 "#PWR01115" H 9450 1750 50  0001 C CNN
 F 1 "+5V" H 9465 2073 50  0000 C CNN
 F 2 "" H 9450 1900 50  0001 C CNN
@@
 	9450 3550 9450 3600
 $Comp
-L 74xx:74LS245 U?
+L 74xx:74LS245 U1107
 U 1 1 6205B0B1
 P 9450 5000
-F 0 "U?" H 9200 5650 50  0000 C CNN
+F 0 "U1107" H 9200 5650 50  0000 C CNN
 F 1 "74LS245" H 9650 5650 50  0000 C CNN
 F 2 "" H 9450 5000 50  0001 C CNN
@@
 $EndComp
 $Comp
-L power:GND #PWR?
+L power:GND #PWR01118
 U 1 1 6205B0B7
 P 9450 5850
-F 0 "#PWR?" H 9450 5600 50  0001 C CNN
+F 0 "#PWR01118" H 9450 5600 50  0001 C CNN
 F 1 "GND" H 9455 5677 50  0000 C CNN
 F 2 "" H 9450 5850 50  0001 C CNN
@@
 $EndComp
 $Comp
-L power:+5V #PWR?
+L power:+5V #PWR01117
 U 1 1 6205B0BD
 P 9450 4150
-F 0 "#PWR?" H 9450 4000 50  0001 C CNN
+F 0 "#PWR01117" H 9450 4000 50  0001 C CNN
 F 1 "+5V" H 9465 4323 50  0000 C CNN
 F 2 "" H 9450 4150 50  0001 C CNN
@@
 	9450 5800 9450 5850
 $Comp
-L 74xx:74LS245 U?
+L 74xx:74LS245 U1105
 U 1 1 620627FF
 P 6450 5000
-F 0 "U?" H 6200 5650 50  0000 C CNN
+F 0 "U1105" H 6200 5650 50  0000 C CNN
 F 1 "74LS245" H 6650 5650 50  0000 C CNN
 F 2 "" H 6450 5000 50  0001 C CNN
@@
 $EndComp
 $Comp
-L power:GND #PWR?
+L power:GND #PWR01112
 U 1 1 62062805
 P 6450 5850
-F 0 "#PWR?" H 6450 5600 50  0001 C CNN
+F 0 "#PWR01112" H 6450 5600 50  0001 C CNN
 F 1 "GND" H 6455 5677 50  0000 C CNN
 F 2 "" H 6450 5850 50  0001 C CNN
@@
 $EndComp
 $Comp
-L power:+5V #PWR?
+L power:+5V #PWR01111
 U 1 1 6206280B
 P 6450 4150
-F 0 "#PWR?" H 6450 4000 50  0001 C CNN
+F 0 "#PWR01111" H 6450 4000 50  0001 C CNN
 F 1 "+5V" H 6465 4323 50  0000 C CNN
 F 2 "" H 6450 4150 50  0001 C CNN
@@
 	8950 3150 8400 3150
 $Comp
-L power:GND #PWR?
+L power:GND #PWR01102
 U 1 1 620ADFFF
 P 3000 2850
-F 0 "#PWR?" H 3000 2600 50  0001 C CNN
+F 0 "#PWR01102" H 3000 2600 50  0001 C CNN
 F 1 "GND" H 3005 2677 50  0000 C CNN
 F 2 "" H 3000 2850 50  0001 C CNN
@@
 $EndComp
 $Comp
-L power:GND #PWR?
+L power:GND #PWR01104
 U 1 1 620BE3B3
 P 3000 5100
-F 0 "#PWR?" H 3000 4850 50  0001 C CNN
+F 0 "#PWR01104" H 3000 4850 50  0001 C CNN
 F 1 "GND" H 3005 4927 50  0000 C CNN
 F 2 "" H 3000 5100 50  0001 C CNN
@@
 $EndComp
 $Comp
-L power:GND #PWR?
+L power:GND #PWR01106
 U 1 1 620BE758
 P 3000 7400
-F 0 "#PWR?" H 3000 7150 50  0001 C CNN
+F 0 "#PWR01106" H 3000 7150 50  0001 C CNN
 F 1 "GND" H 3005 7227 50  0000 C CNN
 F 2 "" H 3000 7400 50  0001 C CNN
@@
 $EndComp
 $Comp
-L power:+5V #PWR?
+L power:+5V #PWR01105
 U 1 1 620BF6CD
 P 3000 5700
-F 0 "#PWR?" H 3000 5550 50  0001 C CNN
+F 0 "#PWR01105" H 3000 5550 50  0001 C CNN
 F 1 "+5V" H 3015 5873 50  0000 C CNN
 F 2 "" H 3000 5700 50  0001 C CNN
@@
 	3000 5700 3000 5750
 $Comp
-L power:+5V #PWR?
+L power:+5V #PWR01101
 U 1 1 620C7ECE
 P 3000 1150
-F 0 "#PWR?" H 3000 1000 50  0001 C CNN
+F 0 "#PWR01101" H 3000 1000 50  0001 C CNN
 F 1 "+5V" H 3015 1323 50  0000 C CNN
 F 2 "" H 3000 1150 50  0001 C CNN
@@
 	3000 1150 3000 1200
 $Comp
-L power:+5V #PWR?
+L power:+5V #PWR01103
 U 1 1 620D938E
 P 3000 3400
-F 0 "#PWR?" H 3000 3250 50  0001 C CNN
+F 0 "#PWR01103" H 3000 3250 50  0001 C CNN
 F 1 "+5V" H 3015 3573 50  0000 C CNN
 F 2 "" H 3000 3400 50  0001 C CNN
@@
 	3000 3400 3000 3450
 $Comp
-L power:GND #PWR?
+L power:GND #PWR01114
 U 1 1 6207A885
 P 8850 5600
-F 0 "#PWR?" H 8850 5350 50  0001 C CNN
+F 0 "#PWR01114" H 8850 5350 50  0001 C CNN
 F 1 "GND" H 8855 5427 50  0000 C CNN
 F 2 "" H 8850 5600 50  0001 C CNN
@@
 $EndComp
 $Comp
-L power:GND #PWR?
+L power:GND #PWR01113
 U 1 1 62073AA8
 P 8850 3350
-F 0 "#PWR?" H 8850 3100 50  0001 C CNN
+F 0 "#PWR01113" H 8850 3100 50  0001 C CNN
 F 1 "GND" H 8855 3177 50  0000 C CNN
 F 2 "" H 8850 3350 50  0001 C CNN
@@
 $EndComp
 $Comp
-L power:GND #PWR?
+L power:GND #PWR01108
 U 1 1 620819B5
 P 5850 5600
-F 0 "#PWR?" H 5850 5350 50  0001 C CNN
+F 0 "#PWR01108" H 5850 5350 50  0001 C CNN
 F 1 "GND" H 5855 5427 50  0000 C CNN
 F 2 "" H 5850 5600 50  0001 C CNN
@@
 $EndComp
 $Comp
-L power:GND #PWR?
+L power:GND #PWR01107
 U 1 1 6204BE6F
 P 5850 3350
-F 0 "#PWR?" H 5850 3100 50  0001 C CNN
+F 0 "#PWR01107" H 5850 3100 50  0001 C CNN
 F 1 "GND" H 5855 3177 50  0000 C CNN
 F 2 "" H 5850 3350 50  0001 C CNN

Commit message: ddraig030: more changes as footprints assigned
Parts:
- U1101, U1102, U1103, U1104, U1105, U1106, U1107: footprint (none) -> Package_DIP:DIP-20_W7.62mm_Socket
Changed lines of the file:
@@
 $Descr A4 11693 8268
 encoding utf-8
-Sheet 13 15
+Sheet 11 16
 Title ""
 Date ""
@@
 F 0 "U1101" H 2750 2650 50  0000 C CNN
 F 1 "74LS241" H 3250 2650 50  0000 C CNN
-F 2 "" H 3000 2000 50  0001 C CNN
+F 2 "Package_DIP:DIP-20_W7.62mm_Socket" H 3000 2000 50  0001 C CNN
 F 3 "http://www.ti.com/lit/ds/symlink/sn74ls241.pdf" H 3000 2000 50  0001 C CNN
 	1    3000 2000
@@
 F 0 "U1102" H 2750 4900 50  0000 C CNN
 F 1 "74LS241" H 3250 4900 50  0000 C CNN
-F 2 "" H 3000 4250 50  0001 C CNN
+F 2 "Package_DIP:DIP-20_W7.62mm_Socket" H 3000 4250 50  0001 C CNN
 F 3 "http://www.ti.com/lit/ds/symlink/sn74ls241.pdf" H 3000 4250 50  0001 C CNN
 	1    3000 4250
@@
 F 0 "U1103" H 2750 7200 50  0000 C CNN
 F 1 "74LS241" H 3250 7200 50  0000 C CNN
-F 2 "" H 3000 6550 50  0001 C CNN
+F 2 "Package_DIP:DIP-20_W7.62mm_Socket" H 3000 6550 50  0001 C CNN
 F 3 "http://www.ti.com/lit/ds/symlink/sn74ls241.pdf" H 3000 6550 50  0001 C CNN
 	1    3000 6550
@@
 F 0 "U1104" H 6200 3400 50  0000 C CNN
 F 1 "74LS245" H 6650 3400 50  0000 C CNN
-F 2 "" H 6450 2750 50  0001 C CNN
+F 2 "Package_DIP:DIP-20_W7.62mm_Socket" H 6450 2750 50  0001 C CNN
 F 3 "http://www.ti.com/lit/gpn/sn74LS245" H 6450 2750 50  0001 C CNN
 	1    6450 2750
@@
 F 0 "U1106" H 9200 3400 50  0000 C CNN
 F 1 "74LS245" H 9650 3400 50  0000 C CNN
-F 2 "" H 9450 2750 50  0001 C CNN
+F 2 "Package_DIP:DIP-20_W7.62mm_Socket" H 9450 2750 50  0001 C CNN
 F 3 "http://www.ti.com/lit/gpn/sn74LS245" H 9450 2750 50  0001 C CNN
 	1    9450 2750
@@
 F 0 "U1107" H 9200 5650 50  0000 C CNN
 F 1 "74LS245" H 9650 5650 50  0000 C CNN
-F 2 "" H 9450 5000 50  0001 C CNN
+F 2 "Package_DIP:DIP-20_W7.62mm_Socket" H 9450 5000 50  0001 C CNN
 F 3 "http://www.ti.com/lit/gpn/sn74LS245" H 9450 5000 50  0001 C CNN
 	1    9450 5000
@@
 F 0 "U1105" H 6200 5650 50  0000 C CNN
 F 1 "74LS245" H 6650 5650 50  0000 C CNN
-F 2 "" H 6450 5000 50  0001 C CNN
+F 2 "Package_DIP:DIP-20_W7.62mm_Socket" H 6450 5000 50  0001 C CNN
 F 3 "http://www.ti.com/lit/gpn/sn74LS245" H 6450 5000 50  0001 C CNN
 	1    6450 5000

Commit message: ddraig030: trying to fix the DRC errors
Connections:
- net +5V: now also U1101.19 (OEb), U1102.19 (OEb), U1103.19 (OEb)
- net GND: now also U1101.1 (OEa), U1101.10 (GND), U1102.1 (OEa), U1102.10 (GND), U1103.1 (OEa), U1103.10 (GND)
- net CAS_A0 renamed ~CAS_A0
- net CAS_A1 renamed ~CAS_A1
- net CAS_A2 renamed ~CAS_A2
- net CAS_A3 renamed ~CAS_A3
- net CAS_B0 renamed ~CAS_B0
- net CAS_B1 renamed ~CAS_B1
- net CAS_B2 renamed ~CAS_B2
- net CAS_B3 renamed ~CAS_B3
