File: yddraig030/DRAM.kicad_sch (KiCad schematic)
At the start: 15 parts, among them U1001 XC95108PQ100, U1002 74LS541, X1001 80Mhz

Commit message: yddraig030: board changed, ready for footprint assignment
Parts:
- removed U1002: 74LS541, Package_DIP:DIP-20_W7.62mm_Socket, symbol 74xx:74LS541
- removed X1001: 80Mhz, Oscillator:Oscillator_DIP-14, symbol Oscillator:ACO-xxxMHz
Connections:
- net RAM_D24 is gone; now on net D24: JSIMM1001.50 (D24), SIMM1001.50 (D24)
- net RAM_D25 is gone; now on net D25: JSIMM1001.52 (D25), SIMM1001.52 (D25)
- net RAM_D26 is gone; now on net D26: JSIMM1001.54 (D26), SIMM1001.54 (D26)
- net RAM_D27 is gone; now on net D27: JSIMM1001.56 (D27), SIMM1001.56 (D27)
- net RAM_D28 is gone; now on net D28: JSIMM1001.58 (D28), SIMM1001.58 (D28)
- net RAM_D29 is gone; now on net D29: JSIMM1001.60 (D29), SIMM1001.60 (D29)
- net RAM_D30 is gone; now on net D30: JSIMM1001.62 (D30), SIMM1001.62 (D30)
- net RAM_D31 is gone; now on net D31: JSIMM1001.64 (D31), SIMM1001.64 (D31)
- net SIM_A0 is gone; now on net MUX_A0: JSIMM1001.12 (A0), SIMM1001.12 (A0)
- net SIM_A1 is gone; now on net MUX_A1: JSIMM1001.13 (A1), SIMM1001.13 (A1)
- net SIM_A10 is gone; now on net MUX_A10: JSIMM1001.19 (A10), SIMM1001.19 (A10)
- net SIM_A11 is gone; now on net MUX_A11: JSIMM1001.29 (A11), SIMM1001.29 (A11)
- net SIM_A2 is gone; now on net MUX_A2: JSIMM1001.14 (A2), SIMM1001.14 (A2)
- net SIM_A3 is gone; now on net MUX_A3: JSIMM1001.15 (A3), SIMM1001.15 (A3)
- net SIM_A4 is gone; now on net MUX_A4: JSIMM1001.16 (A4), SIMM1001.16 (A4)
- net SIM_A5 is gone; now on net MUX_A5: JSIMM1001.17 (A5), SIMM1001.17 (A5)
- net SIM_A6 is gone; now on net MUX_A6: JSIMM1001.18 (A6), SIMM1001.18 (A6)
- net SIM_A7 is gone; now on net MUX_A7: JSIMM1001.28 (A7), SIMM1001.28 (A7)
- net SIM_A8 is gone; now on net MUX_A8: JSIMM1001.31 (A8), SIMM1001.31 (A8)
- net SIM_A9 is gone; now on net MUX_A9: JSIMM1001.32 (A9), SIMM1001.32 (A9)
- net ~{BCAS_A0} is gone; now on net ~{CAS_A0}: SIMM1001.40 (~{CAS0})
- net ~{BCAS_A1} is gone; now on net ~{CAS_A1}: SIMM1001.43 (~{CAS1})
- net ~{BCAS_A2} is gone; now on net ~{CAS_A2}: SIMM1001.41 (~{CAS2})
- net ~{BCAS_A3} is gone; now on net ~{CAS_A3}: SIMM1001.42 (~{CAS3})
- net ~{BCAS_B0} is gone; now on net ~{CAS_B0}: JSIMM1001.40 (~{CAS0})
- net ~{BCAS_B1} is gone; now on net ~{CAS_B1}: JSIMM1001.43 (~{CAS1})
- net ~{BCAS_B2} is gone; now on net ~{CAS_B2}: JSIMM1001.41 (~{CAS2})
- net ~{BCAS_B3} is gone; now on net ~{CAS_B3}: JSIMM1001.42 (~{CAS3})
- net ~{BRAS0} is gone; now on net ~{RAS0}: JSIMM1001.44 (~{RAS0}), SIMM1001.44 (~{RAS0})
- net ~{BRAS1} is gone; now on net ~{RAS1}: JSIMM1001.45 (~{RAS1}), SIMM1001.45 (~{RAS1})
- net ~{BRAS2} is gone; now on net ~{RAS2}: JSIMM1001.34 (~{RAS2}), SIMM1001.34 (~{RAS2})
- net ~{BRAS3} is gone; now on net ~{RAS3}: JSIMM1001.33 (~{RAS3}), SIMM1001.33 (~{RAS3})
- net D24: no longer U1001.82 (P82)
- net D25: no longer U1001.83 (P83)
- net D26: no longer U1001.84 (P84)
- net D27: no longer U1001.87 (P87)
- net D28: no longer U1001.88 (P88)
- net D29: no longer U1001.89 (P89)
- net D30: no longer U1001.91 (P91)
- net D31: no longer U1001.92 (P92)
- net CLK40MHZ: now reaches U1001.24 (I/O/GCK1)
- net RAM_D0 renamed D0
- net RAM_D1 renamed D1
- net RAM_D10 renamed D10
- net RAM_D11 renamed D11
- net RAM_D12 renamed D12
- net RAM_D13 renamed D13
- net RAM_D14 renamed D14
- net RAM_D15 renamed D15
- net RAM_D16 renamed D16
- net RAM_D17 renamed D17
- net RAM_D18 renamed D18
- net RAM_D19 renamed D19
- net RAM_D2 renamed D2
- net RAM_D20 renamed D20
- net RAM_D21 renamed D21
- net RAM_D22 renamed D22
- net RAM_D23 renamed D23
- net RAM_D3 renamed D3
- net RAM_D4 renamed D4
- net RAM_D5 renamed D5
- net RAM_D6 renamed D6
- net RAM_D7 renamed D7
- net RAM_D8 renamed D8
- net RAM_D9 renamed D9
- net ~{CS_DRAMCPLD}: no longer names the net of U1001.94 (P94)
- no-connect marks 12 -> 21
Other:
- removed sheet Buffers
- moved on the sheet: R1001

Commit message: Working on PCB layout
Parts:
- C1001, C1002, C1003, C1004, C1005, C1006, C1007, C1008: footprint Capacitor_THT:C_Disc_D3.8mm_W2.6mm_P2.50mm -> Capacitor_SMD:C_0805_2012Metric
- R1001: footprint Resistor_THT:R_Axial_DIN0207_L6.3mm_D2.5mm_P10.16mm_Horizontal -> Resistor_SMD:R_0805_2012Metric
Changed lines of the file:
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@@
     (property "Reference" "R1001" (id 0) (at 133.35 187.7822 90))
     (property "Value" "22R" (id 1) (at 133.35 190.0936 90))
-    (property "Footprint" "Resistor_THT:R_Axial_DIN0207_L6.3mm_D2.5mm_P10.16mm_Horizontal" (id 2) (at 133.35 191.262 90)
+    (property "Footprint" "Resistor_SMD:R_0805_2012Metric" (id 2) (at 133.35 191.262 90)
       (effects (font (size 1.27 1.27)) hide)
     )
@@
       (effects (font (size 1.27 1.27)) (justify left))
     )
-    (property "Footprint" "Capacitor_THT:C_Disc_D3.8mm_W2.6mm_P2.50mm" (id 2) (at 285.6992 235.585 0)
+    (property "Footprint" "Capacitor_SMD:C_0805_2012Metric" (id 2) (at 285.6992 235.585 0)
       (effects (font (size 1.27 1.27)) hide)
     )
@@
       (effects (font (size 1.27 1.27)) (justify left))
     )
-    (property "Footprint" "Capacitor_THT:C_Disc_D3.8mm_W2.6mm_P2.50mm" (id 2) (at 331.2922 235.331 0)
+    (property "Footprint" "Capacitor_SMD:C_0805_2012Metric" (id 2) (at 331.2922 235.331 0)
       (effects (font (size 1.27 1.27)) hide)
     )
@@
       (effects (font (size 1.27 1.27)) (justify left))
     )
-    (property "Footprint" "Capacitor_THT:C_Disc_D3.8mm_W2.6mm_P2.50mm" (id 2) (at 297.7642 235.585 0)
+    (property "Footprint" "Capacitor_SMD:C_0805_2012Metric" (id 2) (at 297.7642 235.585 0)
       (effects (font (size 1.27 1.27)) hide)
     )
@@
       (effects (font (size 1.27 1.27)) (justify left))
     )
-    (property "Footprint" "Capacitor_THT:C_Disc_D3.8mm_W2.6mm_P2.50mm" (id 2) (at 319.2272 235.331 0)
+    (property "Footprint" "Capacitor_SMD:C_0805_2012Metric" (id 2) (at 319.2272 235.331 0)
       (effects (font (size 1.27 1.27)) hide)
     )
@@
       (effects (font (size 1.27 1.27)) (justify left))
     )
-    (property "Footprint" "Capacitor_THT:C_Disc_D3.8mm_W2.6mm_P2.50mm" (id 2) (at 261.5692 235.585 0)
+    (property "Footprint" "Capacitor_SMD:C_0805_2012Metric" (id 2) (at 261.5692 235.585 0)
       (effects (font (size 1.27 1.27)) hide)
     )
@@
       (effects (font (size 1.27 1.27)) (justify left))
     )
-    (property "Footprint" "Capacitor_THT:C_Disc_D3.8mm_W2.6mm_P2.50mm" (id 2) (at 343.3572 235.331 0)
+    (property "Footprint" "Capacitor_SMD:C_0805_2012Metric" (id 2) (at 343.3572 235.331 0)
       (effects (font (size 1.27 1.27)) hide)
     )
@@
       (effects (font (size 1.27 1.27)) (justify left))
     )
-    (property "Footprint" "Capacitor_THT:C_Disc_D3.8mm_W2.6mm_P2.50mm" (id 2) (at 355.4222 235.331 0)
+    (property "Footprint" "Capacitor_SMD:C_0805_2012Metric" (id 2) (at 355.4222 235.331 0)
       (effects (font (size 1.27 1.27)) hide)
     )
@@
       (effects (font (size 1.27 1.27)) (justify left))
     )
-    (property "Footprint" "Capacitor_THT:C_Disc_D3.8mm_W2.6mm_P2.50mm" (id 2) (at 273.6342 235.585 0)
-      (effects (font (size 1.27 1.27)) hide)
-    )
+    (property "Footprint" "Capacitor_SMD:C_0805_2012Metric" (id 2) (at 273.6342 235.585 0)
+      (effects (font (size 1.27 1.27)) hide)
+    )
