File: yddraig030/RTC.kicad_sch (KiCad schematic)
At the start: 9 parts

Commit message: Updated 030 design files
Parts:
- removed BT?: CR2032, Battery:BatteryHolder_Keystone_103_1x20mm, symbol Device:Battery_Cell
- removed C?: 10uF, Capacitor_THT:CP_Radial_D5.0mm_P2.50mm, symbol Device:CP
- removed D?: 1N4148, Diode_THT:D_DO-35_SOD27_P7.62mm_Horizontal, symbol Diode:1N4148
- removed Q?: BC549B, Package_TO_SOT_THT:TO-92, symbol Device:Q_NPN_EBC
- removed Q?: 2N4403, Package_TO_SOT_THT:TO-92, symbol Device:Q_PNP_EBC
- removed R? (x3): 4K7, Resistor_THT:R_Axial_DIN0207_L6.3mm_D2.5mm_P10.16mm_Horizontal, symbol Device:R
- removed U?: RTC-72421, Package_DIP:DIP-18_W7.62mm_Socket, symbol Ddraig:RTC-72421
- added BT901: CR2032, Battery:BatteryHolder_Keystone_103_1x20mm, symbol Device:Battery_Cell
- added C901: 10uF, Capacitor_THT:CP_Radial_D5.0mm_P2.50mm, symbol Device:C_Polarized
- added D901: 1N4148, Diode_THT:D_DO-35_SOD27_P7.62mm_Horizontal, symbol Diode:1N4148
- added Q901: BC549B, Package_TO_SOT_THT:TO-92, symbol Device:Q_NPN_EBC
- added Q902: 2N4403, Package_TO_SOT_THT:TO-92, symbol Device:Q_PNP_EBC
- added R901, R902, R903: 4K7, Resistor_THT:R_Axial_DIN0207_L6.3mm_D2.5mm_P10.16mm_Horizontal, symbol Device:R
- added U901: RTC-72421, Package_DIP:DIP-18_W7.62mm_Socket, symbol Ddraig:RTC-72421
Connections:
- net +5V: now also Q902.1 (E), R901.1
- net A1: now also U901.4 (A0)
- net A2: now also U901.5 (A1)
- net A3: now also U901.6 (A2)
- net A4: now also U901.7 (A3)
- net D24: now also U901.14 (D0)
- net D25: now also U901.13 (D1)
- net D26: now also U901.12 (D2)
- net D27: now also U901.11 (D3)
- net GND: now also BT901.2 (-), C901.2, Q901.1 (E), R902.2, U901.9 (GND)
- net ~{CS_RTC}: now also U901.2 (~{CS0})
- net ~{RESET}: now also U901.15 (CS1)
- new net: C901.1, D901.1 (K), Q902.3 (C), U901.18 (VDD), U901.3 (ALE)
- new net: Q901.2 (B), R901.2, R902.1
- new net: Q901.3 (C), R903.2
- new net: Q902.2 (B), R903.1
- new net: BT901.1 (+), D901.2 (A)
- new net RD/~{WR}: U901.10 (~{WR})
- new net ~{RD}/WR: U901.8 (~{RD})
Other:
- company: (none) -> Stephen Moody
- title: (none) -> Y Ddraig Fawr

Commit message: More changes to the 030 board
Parts:
- added C? (x2): 100nF, symbol Device:C
Connections:
- net +5V: now also C?.1, C?.1
- net GND: now also C?.2, C?.2
- net RD/~{WR} renamed R/~{W}
- net ~{RD}/WR renamed ~{R}/W
Changed lines of the file:
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@@
   (junction (at 177.8 74.93) (diameter 0) (color 0 0 0 0)
+  )
+  (junction (at 107.188 159.512) (diameter 0) (color 0 0 0 0)
+  )
+  (junction (at 107.823 148.082) (diameter 0) (color 0 0 0 0)
   )
   (junction (at 72.39 74.93) (diameter 0) (color 0 0 0 0)
@@
     (stroke (width 0) (type default) (color 0 0 0 0))
   )
+  (wire (pts (xy 101.473 148.082) (xy 107.823 148.082))
+    (stroke (width 0) (type default) (color 0 0 0 0))
+  )
+  (wire (pts (xy 101.473 148.082) (xy 101.473 149.987))
+    (stroke (width 0) (type default) (color 0 0 0 0))
+  )
   (bus (pts (xy 162.56 99.06) (xy 154.94 99.06))
     (stroke (width 0) (type default) (color 0 0 0 0))
@@
     (stroke (width 0) (type default) (color 0 0 0 0))
   )
+  (wire (pts (xy 101.473 159.512) (xy 107.188 159.512))
+    (stroke (width 0) (type default) (color 0 0 0 0))
+  )
+  (wire (pts (xy 113.538 157.607) (xy 113.538 159.512))
+    (stroke (width 0) (type default) (color 0 0 0 0))
+  )
   (bus (pts (xy 162.56 106.68) (xy 162.56 109.22))
     (stroke (width 0) (type default) (color 0 0 0 0))
@@
     (stroke (width 0) (type default) (color 0 0 0 0))
   )
+  (wire (pts (xy 107.188 159.512) (xy 113.538 159.512))
+    (stroke (width 0) (type default) (color 0 0 0 0))
+  )
   (wire (pts (xy 208.28 104.14) (xy 198.12 104.14))
     (stroke (width 0) (type default) (color 0 0 0 0))
@@
     (stroke (width 0) (type default) (color 0 0 0 0))
   )
+  (wire (pts (xy 107.823 148.082) (xy 113.538 148.082))
+    (stroke (width 0) (type default) (color 0 0 0 0))
+  )
   (wire (pts (xy 172.72 111.76) (xy 165.1 111.76))
     (stroke (width 0) (type default) (color 0 0 0 0))
@@
     (stroke (width 0) (type default) (color 0 0 0 0))
   )
+  (wire (pts (xy 113.538 148.082) (xy 113.538 149.987))
+    (stroke (width 0) (type default) (color 0 0 0 0))
+  )
   (wire (pts (xy 72.39 69.85) (xy 72.39 74.93))
+    (stroke (width 0) (type default) (color 0 0 0 0))
+  )
+  (wire (pts (xy 101.473 157.607) (xy 101.473 159.512))
     (stroke (width 0) (type default) (color 0 0 0 0))
   )
@@
     (effects (font (size 1.27 1.27)) (justify right))
   )
-  (hierarchical_label "~{RD}{slash}WR" (shape input) (at 165.1 116.84 180)
+  (hierarchical_label "~{R}{slash}W" (shape input) (at 165.1 116.84 180)
     (effects (font (size 1.27 1.27)) (justify right))
   )
-  (hierarchical_label "RD{slash}~{WR}" (shape input) (at 165.1 119.38 180)
+  (hierarchical_label "R{slash}~{W}" (shape input) (at 165.1 119.38 180)
     (effects (font (size 1.27 1.27)) (justify right))
   )
@@
     (pin "1")
   )
+  (symbol (lib_id "power:GND") (at 107.188 159.512 0) (unit 1)
+    (in_bom yes) (on_board yes) (fields_autoplaced)
+    (property "Reference" "#PWR?" (id 0) (at 107.188 165.862 0)
+      (effects (font (size 1.27 1.27)) hide)
+    )
+    (property "Value" "GND" (id 1) (at 107.188 164.592 0))
+    (property "Footprint" "" (id 2) (at 107.188 159.512 0)
+      (effects (font (size 1.27 1.27)) hide)
+    )
+    (property "Datasheet" "" (id 3) (at 107.188 159.512 0)
+      (effects (font (size 1.27 1.27)) hide)
+    )
+    (pin "1")
+  )
+  (symbol (lib_id "power:+5V") (at 107.823 148.082 0) (unit 1)
+    (in_bom yes) (on_board yes)
+    (property "Reference" "#PWR?" (id 0) (at 107.823 151.892 0)
+      (effects (font (size 1.27 1.27)) hide)
+    )
+    (property "Value" "+5V" (id 1) (at 108.204 143.6878 0))
+    (property "Footprint" "" (id 2) (at 107.823 148.082 0)
+      (effects (font (size 1.27 1.27)) hide)
+    )
+    (property "Datasheet" "" (id 3) (at 107.823 148.082 0)
+      (effects (font (size 1.27 1.27)) hide)
+    )
+    (pin "1")
+  )
+  (symbol (lib_id "Device:C") (at 113.538 153.797 0) (unit 1)
+    (in_bom yes) (on_board yes) (fields_autoplaced)
+    (property "Reference" "C?" (id 0) (at 116.713 152.5269 0)
+      (effects (font (size 1.27 1.27)) (justify left))
+    )
+    (property "Value" "100nF" (id 1) (at 116.713 155.0669 0)
+      (effects (font (size 1.27 1.27)) (justify left))
+    )
+    (property "Footprint" "" (id 2) (at 114.5032 157.607 0)
+      (effects (font (size 1.27 1.27)) hide)
+    )
+    (property "Datasheet" "~" (id 3) (at 113.538 153.797 0)
+      (effects (font (size 1.27 1.27)) hide)
+    )
+    (pin "1")
+    (pin "2")
+  )
+  (symbol (lib_id "Device:C") (at 101.473 153.797 0) (unit 1)
+    (in_bom yes) (on_board yes) (fields_autoplaced)
+    (property "Reference" "C?" (id 0) (at 104.648 152.5269 0)
+      (effects (font (size 1.27 1.27)) (justify left))
+    )
+    (property "Value" "100nF" (id 1) (at 104.648 155.0669 0)
+      (effects (font (size 1.27 1.27)) (justify left))
+    )
+    (property "Footprint" "" (id 2) (at 102.4382 157.607 0)
+      (effects (font (size 1.27 1.27)) hide)
+    )
+    (property "Datasheet" "~" (id 3) (at 101.473 153.797 0)
+      (effects (font (size 1.27 1.27)) hide)
+    )
+    (pin "1")
+    (pin "2")
+  )
 )

Commit message: ddraig030 schematic done
Parts:
- gave numbers to parts that had none: 2
- renumbered BT901 to BT1401, C901 to C1403, D901 to D1401, Q901 to Q1401, Q902 to Q1402, R901 to R1401, R902 to R1402, R903 to R1403, U901 to U1401
Changed lines of the file:
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@@
   (symbol (lib_id "Ddraig:RTC-72421") (at 185.42 110.49 0) (unit 1)
     (in_bom yes) (on_board yes)
-    (property "Reference" "U901" (id 0) (at 190.5 96.52 0))
+    (property "Reference" "U1401" (id 0) (at 190.5 96.52 0))
     (property "Value" "RTC-72421" (id 1) (at 191.77 127 0))
     (property "Footprint" "Package_DIP:DIP-18_W7.62mm_Socket" (id 2) (at 181.61 109.22 0)
@@
   (symbol (lib_id "Device:Q_NPN_EBC") (at 83.82 100.33 0) (unit 1)
     (in_bom yes) (on_board yes)
-    (property "Reference" "Q901" (id 0) (at 88.6714 99.1616 0)
+    (property "Reference" "Q1401" (id 0) (at 88.6714 99.1616 0)
       (effects (font (size 1.27 1.27)) (justify left))
     )
@@
   (symbol (lib_id "Device:Q_PNP_EBC") (at 86.36 77.47 270) (mirror x) (unit 1)
     (in_bom yes) (on_board yes)
-    (property "Reference" "Q902" (id 0) (at 86.36 69.1388 90))
+    (property "Reference" "Q1402" (id 0) (at 86.36 69.1388 90))
     (property "Value" "2N4403" (id 1) (at 86.36 71.4502 90))
     (property "Footprint" "Package_TO_SOT_THT:TO-92" (id 2) (at 88.9 72.39 0)
@@
   (symbol (lib_id "Diode:1N4148") (at 104.14 82.55 270) (unit 1)
     (in_bom yes) (on_board yes)
-    (property "Reference" "D901" (id 0) (at 106.172 81.3816 90)
+    (property "Reference" "D1401" (id 0) (at 106.172 81.3816 90)
       (effects (font (size 1.27 1.27)) (justify left))
     )
@@
   (symbol (lib_id "Device:Battery_Cell") (at 104.14 93.98 0) (unit 1)
     (in_bom yes) (on_board yes)
-    (property "Reference" "BT901" (id 0) (at 107.1372 91.5416 0)
+    (property "Reference" "BT1401" (id 0) (at 107.1372 91.5416 0)
       (effects (font (size 1.27 1.27)) (justify left))
     )
@@
   (symbol (lib_id "Device:R") (at 72.39 106.68 0) (unit 1)
     (in_bom yes) (on_board yes)
-    (property "Reference" "R902" (id 0) (at 74.168 105.5116 0)
+    (property "Reference" "R1402" (id 0) (at 74.168 105.5116 0)
       (effects (font (size 1.27 1.27)) (justify left))
     )
@@
   (symbol (lib_id "Device:C_Polarized") (at 120.65 87.63 0) (unit 1)
     (in_bom yes) (on_board yes)
-    (property "Reference" "C901" (id 0) (at 123.6472 86.4616 0)
+    (property "Reference" "C1403" (id 0) (at 123.6472 86.4616 0)
       (effects (font (size 1.27 1.27)) (justify left))
     )
@@
   (symbol (lib_id "power:GND") (at 104.14 99.06 0) (unit 1)
     (in_bom yes) (on_board yes)
-    (property "Reference" "#PWR0903" (id 0) (at 104.14 105.41 0)
+    (property "Reference" "#PWR01403" (id 0) (at 104.14 105.41 0)
       (effects (font (size 1.27 1.27)) hide)
     )
@@
   (symbol (lib_id "power:+5V") (at 72.39 69.85 0) (unit 1)
     (in_bom yes) (on_board yes)
-    (property "Reference" "#PWR0901" (id 0) (at 72.39 73.66 0)
+    (property "Reference" "#PWR01401" (id 0) (at 72.39 73.66 0)
       (effects (font (size 1.27 1.27)) hide)
     )
@@
   (symbol (lib_id "power:GND") (at 120.65 99.06 0) (unit 1)
     (in_bom yes) (on_board yes)
-    (property "Reference" "#PWR0904" (id 0) (at 120.65 105.41 0)
+    (property "Reference" "#PWR01406" (id 0) (at 120.65 105.41 0)
       (effects (font (size 1.27 1.27)) hide)
     )
@@
   (symbol (lib_id "Device:R") (at 86.36 88.9 0) (unit 1)
     (in_bom yes) (on_board yes)
-    (property "Reference" "R903" (id 0) (at 88.138 87.7316 0)
+    (property "Reference" "R1403" (id 0) (at 88.138 87.7316 0)
       (effects (font (size 1.27 1.27)) (justify left))
     )
@@
   (symbol (lib_id "Device:R") (at 72.39 88.9 0) (unit 1)
     (in_bom yes) (on_board yes)
-    (property "Reference" "R901" (id 0) (at 74.168 87.7316 0)
+    (property "Reference" "R1401" (id 0) (at 74.168 87.7316 0)
       (effects (font (size 1.27 1.27)) (justify left))
     )
@@
   (symbol (lib_id "power:GND") (at 80.01 114.3 0) (unit 1)
     (in_bom yes) (on_board yes)
-    (property "Reference" "#PWR0902" (id 0) (at 80.01 120.65 0)
+    (property "Reference" "#PWR01402" (id 0) (at 80.01 120.65 0)
       (effects (font (size 1.27 1.27)) hide)
     )
@@
   (symbol (lib_id "power:GND") (at 185.42 132.08 0) (unit 1)
     (in_bom yes) (on_board yes)
-    (property "Reference" "#PWR0905" (id 0) (at 185.42 138.43 0)
+    (property "Reference" "#PWR01407" (id 0) (at 185.42 138.43 0)
       (effects (font (size 1.27 1.27)) hide)
     )
@@
   (symbol (lib_id "power:PWR_FLAG") (at 177.8 74.93 0) (unit 1)
     (in_bom yes) (on_board yes)
-    (property "Reference" "#FLG0901" (id 0) (at 177.8 73.025 0)
+    (property "Reference" "#FLG01401" (id 0) (at 177.8 73.025 0)
       (effects (font (size 1.27 1.27)) hide)
     )
@@
   (symbol (lib_id "power:GND") (at 107.188 159.512 0) (unit 1)
     (in_bom yes) (on_board yes) (fields_autoplaced)
-    (property "Reference" "#PWR?" (id 0) (at 107.188 165.862 0)
+    (property "Reference" "#PWR01404" (id 0) (at 107.188 165.862 0)
       (effects (font (size 1.27 1.27)) hide)
     )
@@
   (symbol (lib_id "power:+5V") (at 107.823 148.082 0) (unit 1)
     (in_bom yes) (on_board yes)
-    (property "Reference" "#PWR?" (id 0) (at 107.823 151.892 0)
+    (property "Reference" "#PWR01405" (id 0) (at 107.823 151.892 0)
       (effects (font (size 1.27 1.27)) hide)
     )
@@
   (symbol (lib_id "Device:C") (at 113.538 153.797 0) (unit 1)
     (in_bom yes) (on_board yes) (fields_autoplaced)
-    (property "Reference" "C?" (id 0) (at 116.713 152.5269 0)
+    (property "Reference" "C1402" (id 0) (at 116.713 152.5269 0)
       (effects (font (size 1.27 1.27)) (justify left))
     )
@@
   (symbol (lib_id "Device:C") (at 101.473 153.797 0) (unit 1)
     (in_bom yes) (on_board yes) (fields_autoplaced)
-    (property "Reference" "C?" (id 0) (at 104.648 152.5269 0)
-      (effects (font (size 1.27 1.27)) (justify left))
-    )
+    (property "Reference" "C1401" (id 0) (at 104.648 152.5269 0)
+      (effects (font (size 1.27 1.27)) (justify left))
+    )

Commit message: Small changes to 030 design
Parts:
- C1401, C1402: footprint (none) -> Capacitor_THT:C_Disc_D3.8mm_W2.6mm_P2.50mm
Changed lines of the file:
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@@
       (effects (font (size 1.27 1.27)) (justify left))
     )
-    (property "Footprint" "" (id 2) (at 114.5032 157.607 0)
+    (property "Footprint" "Capacitor_THT:C_Disc_D3.8mm_W2.6mm_P2.50mm" (id 2) (at 114.5032 157.607 0)
       (effects (font (size 1.27 1.27)) hide)
     )
@@
       (effects (font (size 1.27 1.27)) (justify left))
     )
-    (property "Footprint" "" (id 2) (at 102.4382 157.607 0)
+    (property "Footprint" "Capacitor_THT:C_Disc_D3.8mm_W2.6mm_P2.50mm" (id 2) (at 102.4382 157.607 0)
       (effects (font (size 1.27 1.27)) hide)
     )

Commit message: yddraig030: board changed, ready for footprint assignment
Parts:
- renumbered BT1401 to BT1301, C1401 to C1301, C1402 to C1302, C1403 to C1303, D1401 to D1301, Q1401 to Q1301, Q1402 to Q1302, R1401 to R1301, R1402 to R1302, R1403 to R1303, U1401 to U1301
Changed lines of the file:
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@@
   (symbol (lib_id "Ddraig:RTC-72421") (at 185.42 110.49 0) (unit 1)
     (in_bom yes) (on_board yes)
-    (property "Reference" "U1401" (id 0) (at 190.5 96.52 0))
+    (property "Reference" "U1301" (id 0) (at 190.5 96.52 0))
     (property "Value" "RTC-72421" (id 1) (at 191.77 127 0))
     (property "Footprint" "Package_DIP:DIP-18_W7.62mm_Socket" (id 2) (at 181.61 109.22 0)
@@
   (symbol (lib_id "Device:Q_NPN_EBC") (at 83.82 100.33 0) (unit 1)
     (in_bom yes) (on_board yes)
-    (property "Reference" "Q1401" (id 0) (at 88.6714 99.1616 0)
+    (property "Reference" "Q1301" (id 0) (at 88.6714 99.1616 0)
       (effects (font (size 1.27 1.27)) (justify left))
     )
@@
   (symbol (lib_id "Device:Q_PNP_EBC") (at 86.36 77.47 270) (mirror x) (unit 1)
     (in_bom yes) (on_board yes)
-    (property "Reference" "Q1402" (id 0) (at 86.36 69.1388 90))
+    (property "Reference" "Q1302" (id 0) (at 86.36 69.1388 90))
     (property "Value" "2N4403" (id 1) (at 86.36 71.4502 90))
     (property "Footprint" "Package_TO_SOT_THT:TO-92" (id 2) (at 88.9 72.39 0)
@@
   (symbol (lib_id "Diode:1N4148") (at 104.14 82.55 270) (unit 1)
     (in_bom yes) (on_board yes)
-    (property "Reference" "D1401" (id 0) (at 106.172 81.3816 90)
+    (property "Reference" "D1301" (id 0) (at 106.172 81.3816 90)
       (effects (font (size 1.27 1.27)) (justify left))
     )
@@
   (symbol (lib_id "Device:Battery_Cell") (at 104.14 93.98 0) (unit 1)
     (in_bom yes) (on_board yes)
-    (property "Reference" "BT1401" (id 0) (at 107.1372 91.5416 0)
+    (property "Reference" "BT1301" (id 0) (at 107.1372 91.5416 0)
       (effects (font (size 1.27 1.27)) (justify left))
     )
@@
   (symbol (lib_id "Device:R") (at 72.39 106.68 0) (unit 1)
     (in_bom yes) (on_board yes)
-    (property "Reference" "R1402" (id 0) (at 74.168 105.5116 0)
+    (property "Reference" "R1302" (id 0) (at 74.168 105.5116 0)
       (effects (font (size 1.27 1.27)) (justify left))
     )
@@
   (symbol (lib_id "Device:C_Polarized") (at 120.65 87.63 0) (unit 1)
     (in_bom yes) (on_board yes)
-    (property "Reference" "C1403" (id 0) (at 123.6472 86.4616 0)
+    (property "Reference" "C1303" (id 0) (at 123.6472 86.4616 0)
       (effects (font (size 1.27 1.27)) (justify left))
     )
@@
   (symbol (lib_id "power:GND") (at 104.14 99.06 0) (unit 1)
     (in_bom yes) (on_board yes)
-    (property "Reference" "#PWR01403" (id 0) (at 104.14 105.41 0)
+    (property "Reference" "#PWR01303" (id 0) (at 104.14 105.41 0)
       (effects (font (size 1.27 1.27)) hide)
     )
@@
   (symbol (lib_id "power:+5V") (at 72.39 69.85 0) (unit 1)
     (in_bom yes) (on_board yes)
-    (property "Reference" "#PWR01401" (id 0) (at 72.39 73.66 0)
+    (property "Reference" "#PWR01301" (id 0) (at 72.39 73.66 0)
       (effects (font (size 1.27 1.27)) hide)
     )
@@
   (symbol (lib_id "power:GND") (at 120.65 99.06 0) (unit 1)
     (in_bom yes) (on_board yes)
-    (property "Reference" "#PWR01406" (id 0) (at 120.65 105.41 0)
+    (property "Reference" "#PWR01306" (id 0) (at 120.65 105.41 0)
       (effects (font (size 1.27 1.27)) hide)
     )
@@
   (symbol (lib_id "Device:R") (at 86.36 88.9 0) (unit 1)
     (in_bom yes) (on_board yes)
-    (property "Reference" "R1403" (id 0) (at 88.138 87.7316 0)
+    (property "Reference" "R1303" (id 0) (at 88.138 87.7316 0)
       (effects (font (size 1.27 1.27)) (justify left))
     )
@@
   (symbol (lib_id "Device:R") (at 72.39 88.9 0) (unit 1)
     (in_bom yes) (on_board yes)
-    (property "Reference" "R1401" (id 0) (at 74.168 87.7316 0)
+    (property "Reference" "R1301" (id 0) (at 74.168 87.7316 0)
       (effects (font (size 1.27 1.27)) (justify left))
     )
@@
   (symbol (lib_id "power:GND") (at 80.01 114.3 0) (unit 1)
     (in_bom yes) (on_board yes)
-    (property "Reference" "#PWR01402" (id 0) (at 80.01 120.65 0)
+    (property "Reference" "#PWR01302" (id 0) (at 80.01 120.65 0)
       (effects (font (size 1.27 1.27)) hide)
     )
@@
   (symbol (lib_id "power:GND") (at 185.42 132.08 0) (unit 1)
     (in_bom yes) (on_board yes)
-    (property "Reference" "#PWR01407" (id 0) (at 185.42 138.43 0)
+    (property "Reference" "#PWR01307" (id 0) (at 185.42 138.43 0)
       (effects (font (size 1.27 1.27)) hide)
     )
@@
   (symbol (lib_id "power:PWR_FLAG") (at 177.8 74.93 0) (unit 1)
     (in_bom yes) (on_board yes)
-    (property "Reference" "#FLG01401" (id 0) (at 177.8 73.025 0)
+    (property "Reference" "#FLG01301" (id 0) (at 177.8 73.025 0)
       (effects (font (size 1.27 1.27)) hide)
     )
@@
   (symbol (lib_id "power:GND") (at 107.188 159.512 0) (unit 1)
     (in_bom yes) (on_board yes) (fields_autoplaced)
-    (property "Reference" "#PWR01404" (id 0) (at 107.188 165.862 0)
+    (property "Reference" "#PWR01304" (id 0) (at 107.188 165.862 0)
       (effects (font (size 1.27 1.27)) hide)
     )
@@
   (symbol (lib_id "power:+5V") (at 107.823 148.082 0) (unit 1)
     (in_bom yes) (on_board yes)
-    (property "Reference" "#PWR01405" (id 0) (at 107.823 151.892 0)
+    (property "Reference" "#PWR01305" (id 0) (at 107.823 151.892 0)
       (effects (font (size 1.27 1.27)) hide)
     )
@@
   (symbol (lib_id "Device:C") (at 113.538 153.797 0) (unit 1)
     (in_bom yes) (on_board yes) (fields_autoplaced)
-    (property "Reference" "C1402" (id 0) (at 116.713 152.5269 0)
+    (property "Reference" "C1302" (id 0) (at 116.713 152.5269 0)
       (effects (font (size 1.27 1.27)) (justify left))
     )
@@
   (symbol (lib_id "Device:C") (at 101.473 153.797 0) (unit 1)
     (in_bom yes) (on_board yes) (fields_autoplaced)
-    (property "Reference" "C1401" (id 0) (at 104.648 152.5269 0)
-      (effects (font (size 1.27 1.27)) (justify left))
-    )
+    (property "Reference" "C1301" (id 0) (at 104.648 152.5269 0)
+      (effects (font (size 1.27 1.27)) (justify left))
+    )

Commit message: Working on PCB layout
Parts:
- C1301, C1302: footprint Capacitor_THT:C_Disc_D3.8mm_W2.6mm_P2.50mm -> Capacitor_SMD:C_0805_2012Metric
- C1303: footprint Capacitor_THT:CP_Radial_D5.0mm_P2.50mm -> Capacitor_SMD:CP_Elec_4x5.3
- D1301: footprint Diode_THT:D_DO-35_SOD27_P7.62mm_Horizontal -> Diode_SMD:D_SOD-123
- R1301, R1302, R1303: footprint Resistor_THT:R_Axial_DIN0207_L6.3mm_D2.5mm_P10.16mm_Horizontal -> Resistor_SMD:R_0805_2012Metric
- U1301: footprint Package_DIP:DIP-18_W7.62mm_Socket -> Package_SO:SOP-18_7x12.5mm_P1.27mm
Changed lines of the file:
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@@
     (property "Reference" "U1301" (id 0) (at 190.5 96.52 0))
     (property "Value" "RTC-72421" (id 1) (at 191.77 127 0))
-    (property "Footprint" "Package_DIP:DIP-18_W7.62mm_Socket" (id 2) (at 181.61 109.22 0)
+    (property "Footprint" "Package_SO:SOP-18_7x12.5mm_P1.27mm" (id 2) (at 181.61 109.22 0)
       (effects (font (size 1.27 1.27)) hide)
     )
@@
       (effects (font (size 1.27 1.27)) (justify left))
     )
-    (property "Footprint" "Diode_THT:D_DO-35_SOD27_P7.62mm_Horizontal" (id 2) (at 99.695 82.55 0)
+    (property "Footprint" "Diode_SMD:D_SOD-123" (id 2) (at 99.695 82.55 0)
       (effects (font (size 1.27 1.27)) hide)
     )
@@
       (effects (font (size 1.27 1.27)) (justify left))
     )
-    (property "Footprint" "Resistor_THT:R_Axial_DIN0207_L6.3mm_D2.5mm_P10.16mm_Horizontal" (id 2) (at 70.612 106.68 90)
+    (property "Footprint" "Resistor_SMD:R_0805_2012Metric" (id 2) (at 70.612 106.68 90)
       (effects (font (size 1.27 1.27)) hide)
     )
@@
       (effects (font (size 1.27 1.27)) (justify left))
     )
-    (property "Footprint" "Capacitor_THT:CP_Radial_D5.0mm_P2.50mm" (id 2) (at 121.6152 91.44 0)
+    (property "Footprint" "Capacitor_SMD:CP_Elec_4x5.3" (id 2) (at 121.6152 91.44 0)
       (effects (font (size 1.27 1.27)) hide)
     )
@@
       (effects (font (size 1.27 1.27)) (justify left))
     )
-    (property "Footprint" "Resistor_THT:R_Axial_DIN0207_L6.3mm_D2.5mm_P10.16mm_Horizontal" (id 2) (at 84.582 88.9 90)
+    (property "Footprint" "Resistor_SMD:R_0805_2012Metric" (id 2) (at 84.582 88.9 90)
       (effects (font (size 1.27 1.27)) hide)
     )
@@
       (effects (font (size 1.27 1.27)) (justify left))
     )
-    (property "Footprint" "Resistor_THT:R_Axial_DIN0207_L6.3mm_D2.5mm_P10.16mm_Horizontal" (id 2) (at 70.612 88.9 90)
+    (property "Footprint" "Resistor_SMD:R_0805_2012Metric" (id 2) (at 70.612 88.9 90)
       (effects (font (size 1.27 1.27)) hide)
     )
@@
       (effects (font (size 1.27 1.27)) (justify left))
     )
-    (property "Footprint" "Capacitor_THT:C_Disc_D3.8mm_W2.6mm_P2.50mm" (id 2) (at 114.5032 157.607 0)
+    (property "Footprint" "Capacitor_SMD:C_0805_2012Metric" (id 2) (at 114.5032 157.607 0)
       (effects (font (size 1.27 1.27)) hide)
     )
@@
       (effects (font (size 1.27 1.27)) (justify left))
     )
-    (property "Footprint" "Capacitor_THT:C_Disc_D3.8mm_W2.6mm_P2.50mm" (id 2) (at 102.4382 157.607 0)
-      (effects (font (size 1.27 1.27)) hide)
-    )
+    (property "Footprint" "Capacitor_SMD:C_0805_2012Metric" (id 2) (at 102.4382 157.607 0)
+      (effects (font (size 1.27 1.27)) hide)
+    )
