File: yddraig030/RTC.kicad_sch (KiCad schematic)
At the start: 11 parts, among them Q1301 BC549B, Q1302 2N4403, U1301 RTC-72421

Commit message: Some more changes to SMD version
Parts:
- U1301: footprint Package_SO:SOP-18_7x12.5mm_P1.27mm -> Package_DIP:DIP-18_W7.62mm_Socket
Changed lines of the file:
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@@
     (property "Reference" "U1301" (id 0) (at 190.5 96.52 0))
     (property "Value" "RTC-72421" (id 1) (at 191.77 127 0))
-    (property "Footprint" "Package_SO:SOP-18_7x12.5mm_P1.27mm" (id 2) (at 181.61 109.22 0)
+    (property "Footprint" "Package_DIP:DIP-18_W7.62mm_Socket" (id 2) (at 181.61 109.22 0)
       (effects (font (size 1.27 1.27)) hide)
     )

Commit message: Cleaning up schematic and PCB
Parts:
- D1301: footprint Diode_SMD:D_SOD-123 -> Diode_SMD:D_SOD-323
Other:
- moved on the sheet: C1301, C1302
