File: expansion/AudioYM2151V2/cpu.kicad_sch (KiCad schematic)
At the start: 31 parts, among them J3 JTAG_68K, J4 Serial Out, U10 74LS374, U11 68008, U12 74LS374, U13 74LS148, U14 AS6C4008-55PCN, U15 AT28C256B, U16 XC9536PC44, U17 SC26C92C1A, U9 74LS374, X2 8Mhz, Y1 3.6864Mhz

Commit message: YM2151 board layout progress
Parts:
- added D1: LED, LED_THT:LED_D5.0mm, symbol Device:LED
- added R2: 330R, Resistor_THT:R_Axial_DIN0207_L6.3mm_D2.5mm_P10.16mm_Horizontal, symbol Device:R
- R2: value 220R -> 330R
Connections:
- net +5V: now also D1.2 (A)
- net GND: no longer U9.17 (D6)
- net at U17.14 (OP1): now also R2.2
- new net: D1.1 (K), R2.1
- new net A7: U9.17 (D6)
- no-connect marks 15 -> 14
Changed lines of the file:
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@@
   (junction (at 267.335 242.57) (diameter 0) (color 0 0 0 0)
   )
-  (junction (at 63.5 195.58) (diameter 0) (color 0 0 0 0)
-  )
   (junction (at 267.335 255.27) (diameter 0) (color 0 0 0 0)
   )
@@
   (no_connect (at 140.335 83.82))
   (no_connect (at 353.06 203.2))
-  (no_connect (at 365.76 95.25))
   (no_connect (at 94.615 86.36))
   (no_connect (at 365.76 71.12))
@@
     (stroke (width 0) (type default))
   )
+  (bus_entry (at 53.34 190.5) (size 2.54 2.54)
+    (stroke (width 0) (type default))
+  )
   (bus_entry (at 173.355 58.42) (size 2.54 2.54)
     (stroke (width 0) (type default))
@@
     (stroke (width 0) (type default))
   )
+  (bus (pts (xy 53.34 187.96) (xy 53.34 190.5))
+    (stroke (width 0) (type default))
+  )
   (wire (pts (xy 170.18 162.56) (xy 185.42 162.56))
     (stroke (width 0) (type default))
@@
     (stroke (width 0) (type default))
   )
+  (wire (pts (xy 393.7 71.374) (xy 393.7 73.914))
+    (stroke (width 0) (type default))
+  )
   (wire (pts (xy 61.595 40.64) (xy 61.595 43.18))
     (stroke (width 0) (type default))
@@
     (stroke (width 0) (type default))
   )
-  (wire (pts (xy 63.5 193.04) (xy 68.58 193.04))
-    (stroke (width 0) (type default))
-  )
   (wire (pts (xy 124.46 251.46) (xy 111.76 251.46))
     (stroke (width 0) (type default))
@@
     (stroke (width 0) (type default))
   )
+  (wire (pts (xy 393.7 81.534) (xy 393.7 84.074))
+    (stroke (width 0) (type default))
+  )
   (wire (pts (xy 365.76 110.49) (xy 378.46 110.49))
     (stroke (width 0) (type default))
@@
     (stroke (width 0) (type default))
   )
+  (wire (pts (xy 365.76 95.25) (xy 393.7 95.25))
+    (stroke (width 0) (type default))
+  )
   (wire (pts (xy 272.415 38.1) (xy 272.415 39.37))
     (stroke (width 0) (type default))
@@
     (stroke (width 0) (type default))
   )
+  (wire (pts (xy 55.88 193.04) (xy 68.58 193.04))
+    (stroke (width 0) (type default))
+  )
   (bus (pts (xy 231.775 50.8) (xy 231.775 48.26))
     (stroke (width 0) (type default))
@@
     (stroke (width 0) (type default))
   )
-  (wire (pts (xy 63.5 195.58) (xy 63.5 193.04))
-    (stroke (width 0) (type default))
-  )
   (wire (pts (xy 191.135 48.26) (xy 175.895 48.26))
     (stroke (width 0) (type default))
@@
     (stroke (width 0) (type default))
   )
+  (wire (pts (xy 393.7 91.694) (xy 393.7 95.25))
+    (stroke (width 0) (type default))
+  )
   (wire (pts (xy 216.535 78.74) (xy 226.06 78.74))
     (stroke (width 0) (type default))
@@
     (effects (font (size 1.27 1.27)) (justify right bottom))
   )
+  (label "A7" (at 60.96 193.04 0) (fields_autoplaced)
+    (effects (font (size 1.27 1.27)) (justify left bottom))
+  )
   (label "CPU_A2" (at 144.399 40.64 0) (fields_autoplaced)
     (effects (font (size 1.27 1.27)) (justify left bottom))
@@
     )
   )
+  (symbol (lib_id "Device:R") (at 393.7 87.884 0) (unit 1)
+    (in_bom yes) (on_board yes) (dnp no)
+    (property "Reference" "R2" (at 395.478 86.7156 0)
+      (effects (font (size 1.27 1.27)) (justify left))
+    )
+    (property "Value" "330R" (at 395.478 89.027 0)
+      (effects (font (size 1.27 1.27)) (justify left))
+    )
+    (property "Footprint" "Resistor_THT:R_Axial_DIN0207_L6.3mm_D2.5mm_P10.16mm_Horizontal" (at 391.922 87.884 90)
+      (effects (font (size 1.27 1.27)) hide)
+    )
+    (property "Datasheet" "~" (at 393.7 87.884 0)
+      (effects (font (size 1.27 1.27)) hide)
+    )
+    (pin "1")
+    (pin "2")
+    (instances
+      (project "AudioYM2151V2"
+        (path "/1a0b0354-7e8a-4de9-938d-3a3db9fe7fba"
+          (reference "R2") (unit 1)
+        )
+        (path "/1a0b0354-7e8a-4de9-938d-3a3db9fe7fba/13457701-b9f8-47fd-94fd-78ef7514c622/2383b26c-a42b-4156-bd52-164401cd08a6"
+          (reference "R24") (unit 1)
+        )
+      )
+    )
+  )
   (symbol (lib_id "Device:R") (at 381 87.63 0) (unit 1)
     (in_bom yes) (on_board yes) (dnp no)
@@
       (effects (font (size 1.27 1.27)) (justify left))
     )
-    (property "Value" "220R" (at 382.778 88.773 0)
+    (property "Value" "330R" (at 382.778 88.773 0)
       (effects (font (size 1.27 1.27)) (justify left))
     )
@@
         )
       )
+    )
+  )
+  (symbol (lib_id "Device:LED") (at 393.7 77.724 90) (unit 1)
+    (in_bom yes) (on_board yes) (dnp no)
+    (property "Reference" "D1" (at 396.6972 76.7334 90)
+      (effects (font (size 1.27 1.27)) (justify right))
+    )
+    (property "Value" "LED" (at 396.6972 79.0448 90)
+      (effects (font (size 1.27 1.27)) (justify right))
+    )
+    (property "Footprint" "LED_THT:LED_D5.0mm" (at 393.7 77.724 0)
+      (effects (font (size 1.27 1.27)) hide)
+    )
+    (property "Datasheet" "~" (at 393.7 77.724 0)
+      (effects (font (size 1.27 1.27)) hide)
+    )
+    (pin "1")
+    (pin "2")
+    (instances
+      (project "AudioYM2151V2"
+        (path "/1a0b0354-7e8a-4de9-938d-3a3db9fe7fba"
+          (reference "D1") (unit 1)
+        )
+        (path "/1a0b0354-7e8a-4de9-938d-3a3db9fe7fba/13457701-b9f8-47fd-94fd-78ef7514c622/2383b26c-a42b-4156-bd52-164401cd08a6"
+          (reference "D3") (unit 1)
+        )
+      )
+    )
+  )
+  (symbol (lib_id "power:+5V") (at 393.7 71.374 0) (unit 1)
+    (in_bom yes) (on_board yes) (dnp no)
+    (property "Reference" "#PWR013" (at 393.7 75.184 0)
+      (effects (font (size 1.27 1.27)) hide)
+    )
+    (property "Value" "+5V" (at 393.7 67.818 0)
+      (effects (font (size 1.27 1.27)))
+    )
+    (property "Footprint" "" (at 393.7 71.374 0)
+      (effects (font (size 1.27 1.27)) hide)
+    )
+    (property "Datasheet" "" (at 393.7 71.374 0)
+      (effects (font (size 1.27 1.27)) hide)
+    )
+    (pin "1")
+    (instances
+      (project "AudioYM2151V2"
+        (path "/1a0b0354-7e8a-4de9-938d-3a3db9fe7fba"
+          (reference "#PWR013") (unit 1)
+        )
+        (path "/1a0b0354-7e8a-4de9-938d-3a3db9fe7fba/13457701-b9f8-47fd-94fd-78ef7514c622/2383b26c-a42b-4156-bd52-164401cd08a6"
+          (reference "#PWR0125") (unit 1)
+        )
+      )
