File: expansion/GfxFPGA/VGA.kicad_sch (KiCad schematic)
At the start: 21 parts, among them J501 VGA Out

Commit message: WOrking on VGA card
Parts:
- removed J501: VGA Out, Connector_Dsub:DSUB-15-HD_Female_Horizontal_P2.29x1.98mm_EdgePinOffset3.03mm_Housed_MountingHolesOffset4.94mm, symbol Connector:DB15_Female_HighDensity_MountingHoles
- added J3: DE15_Receptacle_HighDensity, Connector_Dsub:DSUB-15-HD_Female_Horizontal_P2.29x1.98mm_EdgePinOffset3.03mm_Housed_MountingHolesOffset4.94mm, symbol Connector:DE15_Receptacle_HighDensity_MountingHoles
- R21: renamed from R9; footprint (none) -> Resistor_SMD:R_0805_2012Metric
- R22: renamed from R10; footprint (none) -> Resistor_SMD:R_0805_2012Metric
- R23: renamed from R11; footprint (none) -> Resistor_SMD:R_0805_2012Metric
- R24: renamed from R13; footprint (none) -> Resistor_SMD:R_0805_2012Metric
- R25: renamed from R14; footprint (none) -> Resistor_SMD:R_0805_2012Metric
- R26: renamed from R16; footprint (none) -> Resistor_SMD:R_0805_2012Metric
- R27: renamed from R17; footprint (none) -> Resistor_SMD:R_0805_2012Metric
- R28: renamed from R18; footprint (none) -> Resistor_SMD:R_0805_2012Metric
- R29: renamed from R19; footprint (none) -> Resistor_SMD:R_0805_2012Metric
- R30: renamed from R20; footprint (none) -> Resistor_SMD:R_0805_2012Metric
- R31: renamed from R21; footprint (none) -> Resistor_SMD:R_0805_2012Metric
- R32: renamed from R22; footprint (none) -> Resistor_SMD:R_0805_2012Metric
- R33: renamed from R23; footprint (none) -> Resistor_SMD:R_0805_2012Metric
- R34: renamed from R24; footprint (none) -> Resistor_SMD:R_0805_2012Metric
- R35: renamed from R25; footprint (none) -> Resistor_SMD:R_0805_2012Metric
- R36: renamed from R26; footprint (none) -> Resistor_SMD:R_0805_2012Metric
- renumbered C503 to C35, C504 to C36, R504 to R37, R503 to R38
Connections:
- net GND: now also J3.0, J3.10, J3.5, J3.6, J3.7, J3.8
- net HSYNC: now also R37.1; no longer R38.1
- net VSYNC: now also R38.1; no longer R37.1
- net at R38.2: now also J3.14
- net at R37.2: now also J3.13
- net at R21.2, R22.2, R23.2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: now also J3.1
- net at R26.2, R27.2, R28.2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: now also J3.2
- net at R32.2, R33.2, R34.2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: now also J3.3
Other:
- moved on the sheet: R26, R27, R28, R29, R30, R31, R32, R33, R34, R35, R36, R37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
