File: expansion/GfxHDMI/FPGA.kicad_sch (KiCad schematic)
At the start: 30 parts, among them J1 JTAG, U301 XC3S500E-4PQG208I, U302 W25Q64JVSSIM, Y1 ECS-3963

Commit message: Added Spartan-7 FPGA
Parts:
- removed unit 1 of U301
- removed unit 2 of U301
- removed unit 3 of U301
- removed unit 4 of U301
- removed unit 5 of U301
- added U1: XC7S25-CSGA225, Package_BGA:Xilinx_CSGA225, symbol Ddraig:XC7S25-CSGA225
- U302: value W25Q64JVSSIM -> IS25LP064D-JBLE

Commit message: Working on HDMI board
Parts:
- removed U301: XC3S500E-4PQG208I, Ddraig:QFP50P3060X3060X409-208N, symbol Ddraig:XC3S500E-4PQG208I
Connections:
- net D14: no longer U302.2 (DO/IO1)
- net GND: no longer C307.2, C308.2, C309.2, C310.2
- new net: C307.2, C308.2, C309.2, C310.2
- new net FLASH_DO: U302.2 (DO/IO1)
- no-connect marks 18 -> 0
Other:
- moved on the sheet: C1, D1, D2, J1, R1, R10, R11, R12, R2, R3, R301, R302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

Commit message: More work on the HDMI board
Connections:
- net +3V3: now also U1.B7 (VCCO_15), U1.C11 (VCCO_15), U1.C3 (VCCO_34), U1.D5 (VCCBATT_0), U1.E10 (VCCINT), U1.E6 (VCCO_0), U1.E8 (VCCINT), U1.F12 (VCCO_15), U1.F7 (VCCINT), U1.F9 (VCCADC_0), U1.G10 (VCCINT), U1.G2 (VCCO_34), U1.G6 (VCCBRAM), U1.G8 (VREFN_0), U1.H7 (VCCINT), U1.H9 (VREFP_0), U1.J10 (VCCINT), U1.J14 (VCCO_14), U1.J6 (VCCBRAM), U1.K7 (VCCINT), U1.K9 (VCCINT), U1.L3 (VCCO_34), U1.L6 (VCCAUX), U1.L8 (VCCAUX), U1.M12 (VCCO_14), U1.P5 (VCCO_0), U1.P9 (VCCO_14)
- net GND: now also C307.2, C308.2, C309.2, C310.2, U1.A1 (GND), U1.A15 (GND), U1.B8 (GND), U1.C12 (GND), U1.C2 (GND), U1.D14 (GND), U1.D6 (GND), U1.E4 (GND), U1.E7 (GND), U1.E9 (GND), U1.F10 (GND), U1.F13 (GND), U1.F6 (GND), U1.F8 (GNDADC_0), U1.G3 (GND), U1.G7 (GND), U1.H10 (GND), U1.H6 (GND), U1.J13 (GND), U1.J7 (GND), U1.K10 (GND), U1.K6 (GND), U1.K8 (GND), U1.L2 (GND), U1.L7 (GND), U1.L9 (GND), U1.M11 (GND), U1.P13 (GND), U1.P4 (GND), U1.P8 (GND), U1.R1 (GND), U1.R15 (GND)
- net HDMI_TX0_N: now also U1.E15 (IO_L21N_T3_DQS_15)
- net HDMI_TX0_P: now also U1.F14 (IO_L21P_T3_DQS_15)
- net HDMI_TX1_N: now also U1.D15 (IO_L19N_T3_VREF_15)
- net HDMI_TX1_P: now also U1.E14 (IO_L19P_T3_15)
- net HDMI_TX2_N: now also U1.B15 (IO_L14N_T2_SRCC_15)
- net HDMI_TX2_P: now also U1.C15 (IO_L14P_T2_SRCC_15)
- net HDMI_TXC_N: now also U1.F15 (IO_L20N_T3_15)
- net HDMI_TXC_P: now also U1.G15 (IO_L20P_T3_15)
Other:
- moved on the sheet: U1A

Commit message: Added HDMI card based on VGA design
Parts:
- removed R10, R11, R9: 10K, Resistor_SMD:R_0805_2012Metric, symbol Device:R
- removed R3: 390R, Resistor_SMD:R_0805_2012Metric, symbol Device:R
- removed U1: XC7S25-CSGA225, Package_BGA:Xilinx_CSGA225, symbol Ddraig:XC7S25-CSGA225
- added C37: 100nF, Capacitor_SMD:C_0805_2012Metric, symbol Device:C
- added D4: LED, LED_SMD:LED_1206_3216Metric, symbol Device:LED
- added R19: 10K, Resistor_SMD:R_0805_2012Metric, symbol Device:R
- added R6: 390R, Resistor_SMD:R_0805_2012Metric, symbol Device:R
- added U3: XC6SLX9-TQG144, Ddraig:TQ144, symbol FPGA_Xilinx_Spartan6:XC6SLX9-TQG144
- R15: renamed from R1; value 390R -> 10K
- U4: renamed from U302; value IS25LP064D-JBLE -> W25Q64JVSSIM
- renumbered C307 to C10, C308 to C11, C309 to C12, C310 to C13, C301 to C14, C302 to C15, C303 to C16, C304 to C17, C305 to C18, C1 to C19, C306 to C20, D2 to D3, D1 to D5, J1 to J2, R4 to R14, R5 to R16, R6 to R17, R2 to R18, R12 to R5, R301 to R7, R302 to R8, R303 to R9
Connections:
- net ~{ACCESS_LED} is gone; now on net ~{FLASH_CS}: D3.1 (K)
- net +1V2: now also U3.128 (VCCINT), U3.19 (VCCINT), U3.28 (VCCINT), U3.52 (VCCINT), U3.89 (VCCINT)
- net +3V3: now also C37.1, R6.1, U3.103 (VCCO_1), U3.122 (VCCO_0), U3.125 (VCCO_0), U3.129 (VCCAUX), U3.135 (VCCO_0), U3.18 (VCCO_3), U3.20 (VCCAUX), U3.31 (VCCO_3), U3.36 (VCCAUX), U3.4 (VCCO_3), U3.42 (VCCO_2), U3.53 (VCCAUX), U3.63 (VCCO_2), U3.76 (VCCO_1), U3.86 (VCCO_1), U3.90 (VCCAUX)
- net A1: now also U3.41 (IO_L64P_D8_2); no longer R15.1
- net A2: now also U3.43 (IO_L62N_D6_2)
- net A3: now also U3.44 (IO_L62P_D5_2)
- net A4: now also U3.45 (IO_L49N_D4_2)
- net A5: now also U3.46 (IO_L49P_D3_2)
- net A6: now also U3.47 (IO_L48N_RDWR_B_VREF_2)
- net A7: now also U3.48 (IO_L48P_D7_2)
- net A8: now also U3.66 (IO_L2N_CMPMOSI_2)
- net A9: now also U3.67 (IO_L2P_CMPCLK_2)
- net CLK_25MHZ: now also U3.55 (IO_L30N_GCLK0_USERCCLK_2)
- net D0: now also U3.82 (IO_L45N_1)
- net D1: now also U3.83 (IO_L45P_1)
- net D10: now also U3.74 (IO_L74N_DOUT_BUSY_1)
- net D11: now also U3.75 (IO_L74P_AWAKE_1)
- net D12: now also U3.78 (IO_L47N_1)
- net D13: now also U3.79 (IO_L47P_1)
- net D14: now also U3.80 (IO_L46N_1)
- net D15: now also U3.81 (IO_L46P_1); no longer R14.2
- net D2: now also U3.84 (IO_L43N_GCLK4_1)
- net D3: now also U3.85 (IO_L43P_GCLK5_1)
- net D4: now also U3.87 (IO_L42N_GCLK6_TRDY1_1)
- net D5: now also U3.88 (IO_L42P_GCLK7_1)
- net D6: now also U3.92 (IO_L41N_GCLK8_1)
- net D7: now also U3.95 (IO_L40P_GCLK11_1)
- net D8: now also U3.62 (IO_L12P_D1_MISO2_2)
- net D9: now also U3.94 (IO_L40N_GCLK10_1)
- net DATA_DIR: now also U3.59 (IO_L13N_D10_2)
- net FLASH_CLK: now also U3.70 (IO_L1P_CCLK_2)
- net FLASH_DI: now also U3.65 (IO_L3P_D0_DIN_MISO_MISO1_2)
- net FLASH_DO: now also U3.64 (IO_L3N_MOSI_CSI_B_MISO0_2)
- net FPGA_DONE: now also U3.71 (DONE_2)
- net FPGA_INITB: now also U3.39 (IO_L65P_INIT_B_2)
- net FPGA_PROGB: now also U3.37 (PROGRAM_B_2)
- net GND: now also C37.2, R19.2, U3.108 (GND), U3.113 (GND), U3.13 (GND), U3.130 (GND), U3.136 (GND), U3.25 (GND), U3.3 (GND), U3.49 (GND), U3.54 (GND), U3.68 (GND), U3.77 (GND), U3.91 (GND), U3.96 (GND)
- net HDMI_TX0_N: now also U3.99 (IO_L33N_1)
- net HDMI_TX0_P: now also U3.100 (IO_L33P_1)
- net HDMI_TX1_N: now also U3.101 (IO_L32N_1)
- net HDMI_TX1_P: now also U3.102 (IO_L32P_1)
- net HDMI_TX2_N: now also U3.114 (IO_L65N_SCP2_0)
- net HDMI_TX2_P: now also U3.115 (IO_L65P_SCP3_0)
- net HDMI_TXC_N: now also U3.97 (IO_L34N_1)
- net HDMI_TXC_P: now also U3.98 (IO_L34P_1)
- net R~{W}: now also U3.33 (IO_L2P_3)
- net SRAM_A0: now also U3.7 (IO_L51N_3)
- net SRAM_A1: now also U3.6 (IO_L52P_3)
- net SRAM_A10: now also U3.140 (IO_L3P_0)
- net SRAM_A11: now also U3.141 (IO_L2N_0)
- net SRAM_A12: now also U3.142 (IO_L2P_0)
- net SRAM_A13: now also U3.143 (IO_L1N_VREF_0)
- net SRAM_A14: now also U3.144 (IO_L1P_HSWAPEN_0)
- net SRAM_A15: now also U3.27 (IO_L37P_3)
- net SRAM_A16: now also U3.26 (IO_L37N_3)
- net SRAM_A17: now also U3.24 (IO_L41P_GCLK27_3)
- net SRAM_A18: now also U3.23 (IO_L41N_GCLK26_3)
- net SRAM_A19: now also U3.22 (IO_L42P_GCLK25_TRDY2_3)
- net SRAM_A2: now also U3.5 (IO_L52N_3)
- net SRAM_A3: now also U3.2 (IO_L83P_3)
- net SRAM_A4: now also U3.1 (IO_L83N_VREF_3)
- net SRAM_A5: now also U3.117 (IO_L64P_SCP5_0)
- net SRAM_A6: now also U3.118 (IO_L63N_SCP6_0)
- net SRAM_A7: now also U3.119 (IO_L63P_SCP7_0)
- net SRAM_A8: now also U3.120 (IO_L62N_VREF_0)
- net SRAM_A9: now also U3.139 (IO_L3N_0)
- net SRAM_D0: now also U3.9 (IO_L50N_3)
- net SRAM_D1: now also U3.10 (IO_L50P_3)
- net SRAM_D10: now also U3.134 (IO_L34P_GCLK19_0)
- net SRAM_D11: now also U3.133 (IO_L34N_GCLK18_0)
- net SRAM_D12: now also U3.132 (IO_L35P_GCLK17_0)
- net SRAM_D13: now also U3.131 (IO_L35N_GCLK16_0)
- net SRAM_D14: now also U3.127 (IO_L36P_GCLK15_0)
- net SRAM_D15: now also U3.126 (IO_L36N_GCLK14_0)
- net SRAM_D2: now also U3.11 (IO_L49N_3)
- net SRAM_D3: now also U3.12 (IO_L49P_3)
- net SRAM_D4: now also U3.14 (IO_L44N_GCLK20_3)
- net SRAM_D5: now also U3.15 (IO_L44P_GCLK21_3)
- net SRAM_D6: now also U3.16 (IO_L43N_GCLK22_IRDY2_3)
- net SRAM_D7: now also U3.17 (IO_L43P_GCLK23_3)
- net SRAM_D8: now also U3.138 (IO_L4P_0)
- net SRAM_D9: now also U3.137 (IO_L4N_0)
- net ~{AS}: now also U3.61 (IO_L12N_D2_MISO3_2)
- net ~{CPU_DATAEN}: now also U3.58 (IO_L14P_D11_2)
- net ~{CPU_DTACK}: now also U3.50 (IO_L31N_GCLK30_D15_2)
- net ~{CPU_IRQ}: now also U3.51 (IO_L31P_GCLK31_D14_2)
- net ~{DATACS}: now also U3.35 (IO_L1P_3)
- net ~{FLASH_CS}: now also U3.38 (IO_L65N_CSO_B_2)
- net ~{LDS}: now also U3.30 (IO_L36P_3)
- net ~{REGCS}: now also U3.34 (IO_L1N_VREF_3)
- net ~{RESET}: now also U3.29 (IO_L36N_3)
- net ~{SRAM_CS}: now also U3.8 (IO_L51P_3)
- net ~{SRAM_WE}: now also U3.21 (IO_L42N_GCLK24_3)
- net ~{UDS}: now also U3.32 (IO_L2N_3)
- net TCK: now reaches J2.2 (Pin_2)
- net TCK: now also U3.109 (TCK)
- net TDI: now reaches J2.3 (Pin_3)
- net TDI: now also U3.110 (TDI)
- net TDO: now reaches J2.4 (Pin_4)
- net TDO: now also U3.106 (TDO)
- net TMS: now reaches J2.5 (Pin_5)
- net TMS: now also U3.107 (TMS)
- new net: R19.1, U3.73 (SUSPEND)
- new net: D4.2 (A), R6.2
- new net A0: U3.40 (IO_L64N_D9_2)
- new net ADDR_MUX: U3.56 (IO_L30P_GCLK1_D13_2)
- new net FPGA_M0: R14.2, U3.69 (IO_L1N_M0_CMPMISO_2)
- new net FPGA_M1: R15.1, U3.60 (IO_L13P_M1_2)
- new net ~{LED1}: D4.1 (K), U3.57 (IO_L14N_D12_2)
- new net ~{SRAM_LB}: U3.124 (IO_L37P_GCLK13_0)
- new net ~{SRAM_OE}: U3.121 (IO_L62P_0)
- new net ~{SRAM_UB}: U3.123 (IO_L37N_GCLK12_0)
- no-connect marks 0 -> 1
Other:
- moved on the sheet: C19, D3, D5, J2, R14, R15, R16, R17, R18, R5, R7, R8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

Commit message: Changes to the HDMI board
Connections:
- no-connect marks 1 -> 7
Changed lines of the file:
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@@
+	)
+	(no_connect
+		(at 60.96 142.24)
+	)
+	(no_connect
+		(at 162.56 78.74)
+	)
+	(no_connect
+		(at 162.56 104.14)
+	)
+	(no_connect
+		(at 60.96 132.08)
 	)
 	(no_connect
 		(at 331.47 219.71)
 	)
+	(no_connect
+		(at 60.96 139.7)
+	)
+	(no_connect
+		(at 162.56 81.28)
+	)
 	(wire
