File: expansion/GfxHDMI/GfxHDMI.kicad_pcb (KiCad board)
At the start: 4 copper layers, 100 x 100 mm, 90 parts, among them J1 D68K_64PIN_BOARD, J2 JTAG, J4 685119134923, Q1 BC847, U1 SN74LS125ADR, U10 SN74LVC8T245PWR, U11 SN74LVC8T245PWR, U12 SN74LVC8T245PWR, U13 IS61WV102416FBLL-10TLI, U2 LD1117S12TR_SOT223, U3 XC6SLX9-TQG144, U4 W25Q64JVSSIM, U5 SN74LS157NSR, U6 SN74LS157NSR, U7 SN74LS157NSR, U8 SN74LV1T34DBV, U9 SN74LVC8T245PWR, Y1 ECS-3963

Commit message: Changes to the HDMI board
Parts:
- moved C38 45.7 mm to (195.0, 77.3)
- moved C39 44.1 mm to (195.9, 100.3)
- moved C40 4.91 mm to (180.8, 82.0)
- moved C41 4.37 mm to (180.8, 83.7)
- moved C42 4.13 mm to (180.8, 85.3)
- moved C43 3.73 mm to (180.8, 87.0)
- moved C44 3.54 mm to (180.7, 88.6)
- moved C45 3.43 mm to (180.7, 90.3)
- moved C46 3.31 mm to (180.7, 91.9)
- moved C47 3.19 mm to (180.7, 93.6)
- moved D7 1.22 mm to (185.3, 89.4)
- moved D6 1.13 mm to (185.3, 85.8)
- moved R41 0.72 mm to (181.2, 97.8)
- moved R40 0.37 mm to (183.5, 97.8)
- moved J4 0.22 mm to (189.6, 89.0)
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Connections:
- net Net-(C40-Pad2) renamed /HDMI/C_TX2_P
- net Net-(C41-Pad2) renamed /HDMI/C_TX2_N
- net Net-(C42-Pad2) renamed /HDMI/C_TX1_P
- net Net-(C43-Pad2) renamed /HDMI/C_TX1_N
- net Net-(C44-Pad2) renamed /HDMI/C_TX0_P
- net Net-(C45-Pad2) renamed /HDMI/C_TX0_N
- net Net-(C46-Pad2) renamed /HDMI/C_TXC_P
- net Net-(C47-Pad2) renamed /HDMI/C_TXC_N
- net Net-(J4-CLOCK+) renamed /HDMI/TXC_P
- net Net-(J4-CLOCK-) renamed /HDMI/TXC_N
- net Net-(J4-DATA0+) renamed /HDMI/TX0_P
- net Net-(J4-DATA0-) renamed /HDMI/TX0_N
- net Net-(J4-DATA1+) renamed /HDMI/TX1_P
- net Net-(J4-DATA1-) renamed /HDMI/TX1_N
- net Net-(J4-DATA2+) renamed /HDMI/TX2_P
- net Net-(J4-DATA2-) renamed /HDMI/TX2_N
Routing:
- net +5V: track 52.9 -> 101.1 mm
- net /FPGA/D7: track 3.19 -> 49.1 mm
- net /FPGA/~{AS}: track 10.2 -> 50.4 mm, vias 1 -> 2
- net /FPGA/FPGA_M0: track 42.9 -> 3.66 mm, vias 3 -> 1
- net /FPGA/D9: track 4.82 -> 41.3 mm, vias 0 -> 2
- net /FPGA/D8: track 14.1 -> 47.6 mm, vias 1 -> 2
- net /FPGA/FPGA_M1: track 32.2 -> 3.98 mm, vias 3 -> 1
- net /HDMI/HDMI_TX2_P: track 0.00 -> 26.1 mm
- net /HDMI/HDMI_TX2_N: track 0.00 -> 26.0 mm
- net GND: track 138.2 -> 158.8 mm, vias 64 -> 72
- net /FPGA/FLASH_DO: track 53.0 -> 34.3 mm
- net /HDMI/HDMI_TXC_N: track 0.00 -> 17.2 mm
- net /HDMI/HDMI_TXC_P: track 0.00 -> 17.2 mm
- net /HDMI/HDMI_TX1_N: track 0.00 -> 16.5 mm
- net /HDMI/HDMI_TX1_P: track 0.00 -> 16.5 mm
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